Commit message: Moves only linear

File: urdf/gazebo/m2020.gazebo.component_macros.xacro (robot description, xacro)
@@ -43,16 +43,4 @@
        <motorTorqueConstant>${tc}</motorTorqueConstant>
      </transmission>
-<!--      <transmission name="${prefix}_${joint_name}_trans">
-       <type>transmission_interface/SimpleTransmission</type>
-       <joint name="${prefix}_${joint_name}_joint">
-         <hardwareInterface>hardware_interface/EffortJointInterface</hardwareInterface>
-       </joint>
-       <actuator name="${prefix}_${joint_name}_motor">
-         <hardwareInterface>hardware_interface/EffortJointInterface</hardwareInterface>
-         <mechanicalReduction>${reduction}</mechanicalReduction>
-       </actuator>
-       <motorTorqueConstant>${tc}</motorTorqueConstant>
-     </transmission>
-    -->
   </xacro:macro>
   <xacro:macro name="gazebo_dif_drive_trans" params="prefix joint_name reduction tc">
@@ -69,13 +57,18 @@
      </transmission>
   </xacro:macro>
-  <!-- tracbot base xacro -->
-  <!--<xacro:macro name="tracbot_base" params="robot_name side">
-    <xacro:gazebo_dif_drive_trans prefix="${side}" joint_name="wheel" reduction="1" tc="1"/>
-    <xacro:gazebo_simple_trans prefix="front_${side}" joint_name="caster_bracket" reduction="1" tc="1"/>
-    <xacro:gazebo_simple_trans prefix="front_${side}" joint_name="caster_wheel" reduction="1" tc="1"/>
+  <!-- m2020 base xacro -->
+  <xacro:macro name="m2020_base" params="prefix static:=false gravity_off:=true">
+    <xacro:gazebo_dif_drive_trans prefix="${prefix}" joint_name="LF_DRIVE" reduction="1" tc="1"/>
+    <xacro:gazebo_dif_drive_trans prefix="${prefix}" joint_name="LR_DRIVE" reduction="1" tc="1"/>
+    <xacro:gazebo_dif_drive_trans prefix="${prefix}" joint_name="LM_DRIVE" reduction="1" tc="1"/>
+    <xacro:gazebo_dif_drive_trans prefix="${prefix}" joint_name="RF_DRIVE" reduction="1" tc="1"/>
+    <xacro:gazebo_dif_drive_trans prefix="${prefix}" joint_name="RR_DRIVE" reduction="1" tc="1"/>
+    <xacro:gazebo_dif_drive_trans prefix="${prefix}" joint_name="RM_DRIVE" reduction="1" tc="1"/>
+<!--
     <xacro:gazebo_simple_trans prefix="back_${side}" joint_name="caster_bracket" reduction="1" tc="1"/>
     <xacro:gazebo_simple_trans prefix="back_${side}" joint_name="caster_wheel" reduction="1" tc="1"/>
-  </xacro:macro>-->
-  <!-- tracbot arm xacro -->
+  -->
+  </xacro:macro>
+  <!-- m2020 arm xacro -->
   <xacro:macro name="m2020_arm" params="prefix static:=false gravity_off:=true">
     <xacro:gazebo_link prefix="${prefix}" link_name="Body_RA_Link2" collide="true" static="${static}" gravity_off="${gravity_off}"/>

File: urdf/gazebo/m2020.gazebo.components.xacro (robot description, xacro)
@@ -5,5 +5,5 @@
   <xacro:include filename="$(find m2020_urdf_models)/urdf/gazebo/kinect.urdf.xacro"/>
   <!-- build components -->
-  <!--<xacro:m2020_base robot_name="${robot_name}" />-->
+  <xacro:m2020_base prefix="" />
   <xacro:m2020_arm prefix=""/>
   <xacro:m2020_head prefix=""/>

File: urdf/m2020.sim.urdf.xacro (robot description, xacro)
@@ -2,6 +2,81 @@
 <robot name="perseverance" xmlns:xacro="http://www.ros.org/wiki/xacro">
   <xacro:property name="robot_name" value="perseverance" />
+  <xacro:property name="mu1" value="100.0"/>
+  <xacro:property name="mu2" value="100.0"/>
   <xacro:include filename="$(find m2020_urdf_models)/urdf/m2020.traclabs.urdf.xacro" />
   <xacro:include filename="$(find m2020_urdf_models)/urdf/gazebo/m2020.gazebo.components.xacro" />
   <xacro:include filename="$(find m2020_urdf_models)/urdf/gazebo/m2020.gazebo.controllers.xacro" />
+  <!-- Parameters wheels -->
+  <gazebo reference="LF_DRIVE">
+    <implicitSpringDamper>1</implicitSpringDamper>
+  </gazebo>
+  <gazebo reference="LM_DRIVE">
+    <implicitSpringDamper>1</implicitSpringDamper>
+  </gazebo>
+  <gazebo reference="LR_DRIVE">
+    <implicitSpringDamper>1</implicitSpringDamper>
+  </gazebo>
+  <gazebo reference="RF_DRIVE">
+    <implicitSpringDamper>1</implicitSpringDamper>
+  </gazebo>
+  <gazebo reference="RM_DRIVE">
+    <implicitSpringDamper>1</implicitSpringDamper>
+  </gazebo>
+  <gazebo reference="RR_DRIVE">
+    <implicitSpringDamper>1</implicitSpringDamper>
+  </gazebo>
+  <gazebo reference="Body_WheelLeftFront">
+    <kp>1000000.0</kp>
+    <kd>100.0</kd>
+    <mu1>${mu1}</mu1>
+    <mu2>${mu2}</mu2>
+    <!-- <fdir1>1 0 0</fdir1 -->
+    <maxVel>1.0</maxVel>
+    <minDepth>0.01</minDepth>
+  </gazebo>
+  <gazebo reference="Body_WheelLeftRear">
+    <kp>1000000.0</kp>
+    <kd>100.0</kd>
+    <mu1>${mu1}</mu1>
+    <mu2>${mu2}</mu2>
+    <!-- <fdir1>1 0 0</fdir1 -->
+    <maxVel>1.0</maxVel>
+    <minDepth>0.01</minDepth>
+  </gazebo>
+  <gazebo reference="Body_WheelLeftMiddle">
+    <kp>1000000.0</kp>
+    <kd>100.0</kd>
+    <mu1>${mu1}</mu1>
+    <mu2>${mu2}</mu2>
+    <!-- <fdir1>1 0 0</fdir1 -->
+    <maxVel>1.0</maxVel>
+    <minDepth>0.01</minDepth>
+  </gazebo>
+  <gazebo reference="Body_WheelRightFront">
+    <kp>1000000.0</kp>
+    <kd>100.0</kd>
+    <mu1>${mu1}</mu1>
+    <mu2>${mu2}</mu2>
+    <!-- <fdir1>1 0 0</fdir1 -->
+    <maxVel>1.0</maxVel>
+    <minDepth>0.01</minDepth>
+  </gazebo>
+  <gazebo reference="Body_WheelRightRear">
+    <kp>1000000.0</kp>
+    <kd>100.0</kd>
+    <mu1>${mu1}</mu1>
+    <mu2>${mu2}</mu2>
+    <!-- <fdir1>1 0 0</fdir1 -->
+    <maxVel>1.0</maxVel>
+    <minDepth>0.01</minDepth>
+  </gazebo>
+  <gazebo reference="Body_WheelRightMiddle">
+    <kp>1000000.0</kp>
+    <kd>100.0</kd>
+    <mu1>${mu1}</mu1>
+    <mu2>${mu2}</mu2>
+    <!-- <fdir1>1 0 0</fdir1 -->
+    <maxVel>1.0</maxVel>
+    <minDepth>0.01</minDepth>
+  </gazebo>
 </robot>

File: urdf/m2020.traclabs.urdf.xacro (robot description, xacro)
@@ -4,5 +4,7 @@
 <robot name="perseverance" xmlns:xacro="http://www.ros.org/wiki/xacro">
   <!-- TRACLABS NOTES CONVERSION: Commented out: 	<link name="Body_CorerFeed"> CHECK OUT LATER!  -->
+  <!-- Set wheel MIDDLE links to be smaller, so they don't touch the floor (so we only use the front and back for diff driving)-->
   <xacro:include filename="$(find m2020_urdf_models)/urdf/gazebo/m2020.gazebo.component_macros.xacro"/>
+  <xacro:property name="M_PI" value="3.14159"/>
   <xacro:property name="arm_joint_vel" value="0.2" /> <!-- original value: 1.79769e+308 -->
   <xacro:property name="head_joint_vel" value="1.0" /> <!-- original value: 1.79769e+308 -->
@@ -42,4 +44,9 @@
   <xacro:property name="head_friction" value="10.0"/>
   <xacro:property name="head_effort" value="100.0" />
+  <xacro:property name="wheel_mass" value="10.0" />
+  <xacro:property name="wheel_effort" value="1000.0" />
+  <xacro:property name="wheel_velocity" value="20.0" />
+  <xacro:property name="wheel_radius" value="0.255" />
+  <xacro:property name="wheel_width" value="0.331" />
 	<link name="base_footprint"/>
 	<link name="Body_Chassis">
@@ -79,5 +86,5 @@
 	<link name="Body_Differential">
 		<inertial>
-			<origin xyz="0.142 0 0" rpy="0 -0 0"/>
+			<origin xyz="0 0 0" rpy="0 -0 0"/>
 			<mass value="${default_mass}"/>
 			<inertia ixx="${default_ixx}" ixy="0" ixz="0" iyy="${default_iyy}" iyz="0" izz="${default_izz}"/>
@@ -98,5 +105,5 @@
 	<link name="Body_RockerLeft">
 		<inertial>
-			<origin xyz="-0.214 0.79959 -0.2405" rpy="0 -0 0"/>
+			<origin xyz="0 0 0" rpy="0 -0 0"/>
 			<mass value="${default_mass}"/>
 			<inertia ixx="${default_ixx}" ixy="0" ixz="0" iyy="${default_iyy}" iyz="0" izz="${default_izz}"/>
@@ -117,5 +124,5 @@
 	<link name="Body_BogieLeft">
 		<inertial>
-			<origin xyz="0.54 0.91959 -0.4705" rpy="0 -0 0"/>
+			<origin xyz="0.0 0 0" rpy="0 -0 0"/>
 			<mass value="${default_mass}"/>
 			<inertia ixx="${default_ixx}" ixy="0" ixz="0" iyy="${default_iyy}" iyz="0" izz="${default_izz}"/>
@@ -136,5 +143,5 @@
 	<link name="Body_SteerLeftRear">
 		<inertial>
-			<origin xyz="1.165 1.0625 -0.8705" rpy="0 -0 0"/>
+			<origin xyz="0 0 0" rpy="0 -0 0"/>
 			<mass value="${default_mass}"/>
 			<inertia ixx="${default_ixx}" ixy="0" ixz="0" iyy="${default_iyy}" iyz="0" izz="${default_izz}"/>
@@ -155,6 +162,6 @@
 	<link name="Body_WheelLeftRear">
 		<inertial>
-			<origin xyz="1.165 1.0625 -0.8705" rpy="0 -0 0"/>
-			<mass value="${default_mass}"/>
+			<origin xyz="0 0 0" rpy="0 -0 0"/>
+			<mass value="${wheel_mass}"/>
 			<inertia ixx="${default_ixx}" ixy="0" ixz="0" iyy="${default_iyy}" iyz="0" izz="${default_izz}"/>
 		</inertial>
@@ -166,14 +173,18 @@
 		</visual>
 		<collision name="ColGeom_Wheel_LeftRear">
-			<origin xyz="1.165 1.0625 -0.8705" rpy="0 -0 0"/>
+          <origin xyz="0 0 0" rpy="${M_PI/2} 0 0" />
+          <geometry>
+            <cylinder radius="${wheel_radius-0.0001}" length="${wheel_width}"/>
+          </geometry>
+			<!--<origin xyz="1.165 1.0625 -0.8705" rpy="0 -0 0"/>
 			<geometry>
 				<mesh filename="package://m2020_urdf_models/rover/meshes/Wheel_LeftRear.dae" scale="1 1 1"/>
-			</geometry>
+			</geometry>-->
 		</collision>
 	</link>
 	<link name="Body_WheelLeftMiddle">
 		<inertial>
-			<origin xyz="0.09002 1.1845 -0.8705" rpy="0 -0 0"/>
-			<mass value="${default_mass}"/>
+			<origin xyz="0 0 0" rpy="0 -0 0"/>
+			<mass value="${wheel_mass}"/>
 			<inertia ixx="${default_ixx}" ixy="0" ixz="0" iyy="${default_iyy}" iyz="0" izz="${default_izz}"/>
 		</inertial>
@@ -185,8 +196,12 @@
 		</visual>
 		<collision name="ColGeom_Wheel_LeftMiddle">
-			<origin xyz="0.09002 1.1845 -0.8705" rpy="0 -0 0"/>
+          <origin xyz="0 0 0" rpy="${M_PI/2} 0 0" />
+          <geometry>
+            <cylinder radius="${wheel_radius-0.0001}" length="${wheel_width}"/>
+          </geometry>
+			<!--<origin xyz="0.09002 1.1845 -0.8705" rpy="0 -0 0"/>
 			<geometry>
 				<mesh filename="package://m2020_urdf_models/rover/meshes/Wheel_LeftMiddle.dae" scale="1 1 1"/>
-			</geometry>
+			</geometry>-->
 		</collision>
 	</link>
@@ -212,6 +227,6 @@
 	<link name="Body_WheelLeftFront">
 		<inertial>
-			<origin xyz="-1.095 1.0625 -0.8705" rpy="0 -0 0"/>
-			<mass value="${default_mass}"/>
+			<origin xyz="0 0 0" rpy="0 -0 0"/>
+			<mass value="${wheel_mass}"/>
 			<inertia ixx="${default_ixx}" ixy="0" ixz="0" iyy="${default_iyy}" iyz="0" izz="${default_izz}"/>
 		</inertial>
@@ -223,8 +238,12 @@
 		</visual>
 		<collision name="ColGeom_Wheel_LeftFront">
-			<origin xyz="-1.095 1.0625 -0.8705" rpy="0 -0 0"/>
+          <origin xyz="0 0 0" rpy="${M_PI/2} 0 0" />
+          <geometry>
+            <cylinder radius="${wheel_radius-0.0001}" length="${wheel_width}"/>
+          </geometry>
+			<!--<origin xyz="-1.095 1.0625 -0.8705" rpy="0 -0 0"/>
 			<geometry>
 				<mesh filename="package://m2020_urdf_models/rover/meshes/Wheel_LeftFront.dae" scale="1 1 1"/>
-			</geometry>
+			</geometry>-->
 		</collision>
 	</link>
@@ -288,6 +307,6 @@
 	<link name="Body_WheelRightRear">
 		<inertial>
-			<origin xyz="1.165 -1.0625 -0.8705" rpy="0 -0 0"/>
-			<mass value="${default_mass}"/>
+			<origin xyz="0 0 0" rpy="0 -0 0"/>
+			<mass value="${wheel_mass}"/>
 			<inertia ixx="${default_ixx}" ixy="0" ixz="0" iyy="${default_iyy}" iyz="0" izz="${default_izz}"/>
 		</inertial>
@@ -299,14 +318,18 @@
 		</visual>
 		<collision name="ColGeom_Wheel_RightRear">
-			<origin xyz="1.165 -1.0625 -0.8705" rpy="0 -0 0"/>
+          <origin xyz="0 0 0" rpy="${M_PI/2} 0 0" />
+          <geometry>
+            <cylinder radius="${wheel_radius-0.0001}" length="${wheel_width}"/>
+          </geometry>
+			<!--<origin xyz="1.165 -1.0625 -0.8705" rpy="0 -0 0"/>
 			<geometry>
 				<mesh filename="package://m2020_urdf_models/rover/meshes/Wheel_RightRear.dae" scale="1 1 1"/>
-			</geometry>
+			</geometry>-->
 		</collision>
 	</link>
 	<link name="Body_WheelRightMiddle">
 		<inertial>
-			<origin xyz="0.09002 -1.1845 -0.8705" rpy="0 -0 0"/>
-			<mass value="${default_mass}"/>
+			<origin xyz="0 0 0" rpy="0 -0 0"/>
+			<mass value="${wheel_mass}"/>
 			<inertia ixx="${default_ixx}" ixy="0" ixz="0" iyy="${default_iyy}" iyz="0" izz="${default_izz}"/>
 		</inertial>
@@ -318,8 +341,12 @@
 		</visual>
 		<collision name="ColGeom_Wheel_RightMiddle">
-			<origin xyz="0.09002 -1.1845 -0.8705" rpy="0 -0 0"/>
+          <origin xyz="0 0 0" rpy="${M_PI/2} 0 0" />
+          <geometry>
+            <cylinder radius="${wheel_radius-0.0001}" length="${wheel_width}"/>
+          </geometry>
+		  <!--<origin xyz="0.09002 -1.1845 -0.8705" rpy="0 -0 0"/>
 			<geometry>
 				<mesh filename="package://m2020_urdf_models/rover/meshes/Wheel_RightMiddle.dae" scale="1 1 1"/>
-			</geometry>
+			</geometry>-->
 		</collision>
 	</link>
@@ -345,6 +372,6 @@
 	<link name="Body_WheelRightFront">
 		<inertial>
-			<origin xyz="-1.095 -1.0625 -0.8705" rpy="0 -0 0"/>
-			<mass value="${default_mass}"/>
+			<origin xyz="0 0 0" rpy="0 -0 0"/>
+			<mass value="${wheel_mass}"/>
 			<inertia ixx="${default_ixx}" ixy="0" ixz="0" iyy="${default_iyy}" iyz="0" izz="${default_izz}"/>
 		</inertial>
@@ -356,8 +383,12 @@
 		</visual>
 		<collision name="ColGeom_Wheel_RightFront">
-			<origin xyz="-1.095 -1.0625 -0.8705" rpy="0 -0 0"/>
+          <origin xyz="0 0 0" rpy="${M_PI/2} 0 0" />
+          <geometry>
+            <cylinder radius="${wheel_radius-0.0001}" length="${wheel_width}"/>
+          </geometry>
+			<!--<origin xyz="-1.095 -1.0625 -0.8705" rpy="0 -0 0"/>
 			<geometry>
 				<mesh filename="package://m2020_urdf_models/rover/meshes/Wheel_RightFront.dae" scale="1 1 1"/>
-			</geometry>
+			</geometry>-->
 		</collision>
 	</link>
@@ -798,17 +829,19 @@
 		<limit lower="-1.79769e+308" upper="1.79769e+308" effort="1.79769e+308" velocity="1.79769e+308"/>
 	</joint>
-	<joint name="LR_DRIVE" type="fixed"> <!-- TRACLabs Gazebo test hack -->
+	<joint name="LR_DRIVE" type="continuous"> <!-- revolute TRACLabs Gazebo test hack -->
 		<origin xyz="0 0 0" rpy="0 -0 0"/>
 		<parent link="Body_SteerLeftRear"/>
 		<child link="Body_WheelLeftRear"/>
 		<axis xyz="0 -1 0"/>
-		<limit lower="-1.79769e+308" upper="1.79769e+308" effort="1.79769e+308" velocity="1.79769e+308"/>
-	</joint>
-	<joint name="LM_DRIVE" type="fixed"> <!-- TRACLabs Gazebo test hack -->
+		<limit effort="${wheel_effort}" velocity="${wheel_velocity}"/>
+		<dynamics damping="0.0" friction="0.0" />
+	</joint>
+	<joint name="LM_DRIVE" type="continuous"> <!-- revolute TRACLabs Gazebo test hack -->
 		<origin xyz="0.44998 -0.26491 0.4" rpy="0 -0 0"/>
 		<parent link="Body_BogieLeft"/>
 		<child link="Body_WheelLeftMiddle"/>
 		<axis xyz="0 -1 0"/>
-		<limit lower="-1.79769e+308" upper="1.79769e+308" effort="1.79769e+308" velocity="1.79769e+308"/>
+		<limit effort="${wheel_effort}" velocity="${wheel_velocity}"/>
+		<dynamics damping="0.0" friction="0.0" />
 	</joint>
 	<joint name="LF_STEER" type="fixed"> <!-- TRACLabs Gazebo test hack -->
@@ -819,10 +852,11 @@
 		<limit lower="-1.79769e+308" upper="1.79769e+308" effort="1.79769e+308" velocity="1.79769e+308"/>
 	</joint>
-	<joint name="LF_DRIVE" type="fixed"> <!-- TRACLabs Gazebo test hack -->
+	<joint name="LF_DRIVE" type="continuous"> <!-- revolute TRACLabs Gazebo test hack -->
 		<origin xyz="0 0 0" rpy="0 -0 0"/>
 		<parent link="Body_SteerLeftFront"/>
 		<child link="Body_WheelLeftFront"/>
 		<axis xyz="0 -1 0"/>
-		<limit lower="-1.79769e+308" upper="1.79769e+308" effort="1.79769e+308" velocity="1.79769e+308"/>
+		<limit effort="${wheel_effort}" velocity="${wheel_velocity}"/>
+		<dynamics damping="0.0" friction="0.0" />
 	</joint>
 	<joint name="RIGHT_DIFFERENTIAL" type="fixed"> <!-- TRACLabs Gazebo test hack -->
@@ -840,5 +874,5 @@
 		<limit lower="-1.79769e+308" upper="1.79769e+308" effort="1.79769e+308" velocity="1.79769e+308"/>
 	</joint>
-	<joint name="RR_STEER" type="fixed"> <!-- TRACLabs Gazebo test hack -->
+	<joint name="RR_STEER" type="fixed"> <!-- revolute TRACLabs Gazebo test hack -->
 		<origin xyz="-0.625 0.14291 0.4" rpy="0 -0 0"/>
 		<parent link="Body_BogieRight"/>
@@ -847,17 +881,19 @@
 		<limit lower="-1.79769e+308" upper="1.79769e+308" effort="1.79769e+308" velocity="1.79769e+308"/>
 	</joint>
-	<joint name="RR_DRIVE" type="fixed"> <!-- TRACLabs Gazebo test hack -->
+	<joint name="RR_DRIVE" type="continuous">  <!-- revolute TRACLabs Gazebo test hack -->
 		<origin xyz="0 0 0" rpy="0 -0 0"/>
 		<parent link="Body_SteerRightRear"/>
 		<child link="Body_WheelRightRear"/>
 		<axis xyz="0 -1 0"/>
-		<limit lower="-1.79769e+308" upper="1.79769e+308" effort="1.79769e+308" velocity="1.79769e+308"/>
-	</joint>
-	<joint name="RM_DRIVE" type="fixed"> <!-- TRACLabs Gazebo test hack -->
+		<limit effort="${wheel_effort}" velocity="${wheel_velocity}"/>
+		<dynamics damping="0.0" friction="0.0" />
+	</joint>
+	<joint name="RM_DRIVE" type="continuous"> <!-- revolute TRACLabs Gazebo test hack -->
 		<origin xyz="0.44998 0.26491 0.4" rpy="0 -0 0"/>
 		<parent link="Body_BogieRight"/>
 		<child link="Body_WheelRightMiddle"/>
 		<axis xyz="0 -1 0"/>
-		<limit lower="-1.79769e+308" upper="1.79769e+308" effort="1.79769e+308" velocity="1.79769e+308"/>
+		<limit effort="${wheel_effort}" velocity="${wheel_velocity}"/>
+		<dynamics damping="0.0" friction="0.0" />
 	</joint>
 	<joint name="RF_STEER" type="fixed"> <!-- TRACLabs Gazebo test hack -->
@@ -868,10 +904,11 @@
 		<limit lower="-1.79769e+308" upper="1.79769e+308" effort="1.79769e+308" velocity="1.79769e+308"/>
 	</joint>
-	<joint name="RF_DRIVE" type="fixed"> <!-- revolute TRACLabs Gazebo test hack -->
+	<joint name="RF_DRIVE" type="continuous">  <!-- revolute TRACLabs Gazebo test hack -->
 		<origin xyz="0 0 0" rpy="0 -0 0"/>
 		<parent link="Body_SteerRightFront"/>
 		<child link="Body_WheelRightFront"/>
 		<axis xyz="0 -1 0"/>
-		<limit lower="-1.79769e+308" upper="1.79769e+308" effort="1.79769e+308" velocity="1.79769e+308"/>
+		<limit effort="${wheel_effort}" velocity="${wheel_velocity}"/>
+		<dynamics damping="0.0" friction="0.0" />
 	</joint>
 	<joint name="RSM_AZ_ENC" type="revolute">
