Commit message: Robot can rotate, love you Perseverance

File: urdf/gazebo/m2020.gazebo.component_macros.xacro (robot description, xacro)
@@ -65,4 +65,5 @@
     <xacro:gazebo_dif_drive_trans prefix="${prefix}" joint_name="RR_DRIVE" reduction="1" tc="1"/>
     <xacro:gazebo_dif_drive_trans prefix="${prefix}" joint_name="RM_DRIVE" reduction="1" tc="1"/>
+    <xacro:gazebo_link prefix="${prefix}" link_name="Body_Chassis" collide="true" static="${static}" gravity_off="${gravity_off}"/>
 <!--
     <xacro:gazebo_simple_trans prefix="back_${side}" joint_name="caster_bracket" reduction="1" tc="1"/>

File: urdf/m2020.sim.urdf.xacro (robot description, xacro)
@@ -31,5 +31,5 @@
     <mu1>${mu1}</mu1>
     <mu2>${mu2}</mu2>
-    <!-- <fdir1>1 0 0</fdir1 -->
+    <fdir1>1 0 0</fdir1>
     <maxVel>1.0</maxVel>
     <minDepth>0.01</minDepth>
@@ -40,5 +40,5 @@
     <mu1>${mu1}</mu1>
     <mu2>${mu2}</mu2>
-    <!-- <fdir1>1 0 0</fdir1 -->
+    <fdir1>1 0 0</fdir1>
     <maxVel>1.0</maxVel>
     <minDepth>0.01</minDepth>

File: urdf/m2020.traclabs.urdf.xacro (robot description, xacro)
@@ -7,5 +7,5 @@
   <xacro:include filename="$(find m2020_urdf_models)/urdf/gazebo/m2020.gazebo.component_macros.xacro"/>
   <xacro:property name="M_PI" value="3.14159"/>
-  <xacro:property name="arm_joint_vel" value="0.2" /> <!-- original value: 1.79769e+308 -->
+  <xacro:property name="arm_joint_vel" value="0.6" /> <!-- original value: 1.79769e+308 -->
   <xacro:property name="head_joint_vel" value="1.0" /> <!-- original value: 1.79769e+308 -->
   <xacro:property name="arm_default_effort" value="100.0" /> <!-- original value: 1.79769e+308 -->
@@ -45,4 +45,7 @@
   <xacro:property name="head_effort" value="100.0" />
   <xacro:property name="wheel_mass" value="10.0" />
+  <xacro:property name="wheel_ixx" value="${0.0254*wheel_mass}" />
+  <xacro:property name="wheel_iyy" value="${0.0325*wheel_mass}" />
+  <xacro:property name="wheel_izz" value="${0.0254*wheel_mass}" />
   <xacro:property name="wheel_effort" value="1000.0" />
   <xacro:property name="wheel_velocity" value="20.0" />
@@ -162,7 +165,7 @@
 	<link name="Body_WheelLeftRear">
 		<inertial>
-			<origin xyz="0 0 0" rpy="0 -0 0"/>
+			<origin xyz="0 0 0" rpy="0 0 0"/>
 			<mass value="${wheel_mass}"/>
-			<inertia ixx="${default_ixx}" ixy="0" ixz="0" iyy="${default_iyy}" iyz="0" izz="${default_izz}"/>
+			<inertia ixx="${wheel_ixx}" ixy="0" ixz="0" iyy="${wheel_iyy}" iyz="0" izz="${wheel_izz}"/>
 		</inertial>
 		<visual name="VisGeom_Wheel_LeftRear">
@@ -177,8 +180,4 @@
             <cylinder radius="${wheel_radius-0.0001}" length="${wheel_width}"/>
           </geometry>
-			<!--<origin xyz="1.165 1.0625 -0.8705" rpy="0 -0 0"/>
-			<geometry>
-				<mesh filename="package://m2020_urdf_models/rover/meshes/Wheel_LeftRear.dae" scale="1 1 1"/>
-			</geometry>-->
 		</collision>
 	</link>
@@ -187,5 +186,5 @@
 			<origin xyz="0 0 0" rpy="0 -0 0"/>
 			<mass value="${wheel_mass}"/>
-			<inertia ixx="${default_ixx}" ixy="0" ixz="0" iyy="${default_iyy}" iyz="0" izz="${default_izz}"/>
+			<inertia ixx="${wheel_ixx}" ixy="0" ixz="0" iyy="${wheel_iyy}" iyz="0" izz="${wheel_izz}"/>
 		</inertial>
 		<visual name="VisGeom_Wheel_LeftMiddle">
@@ -200,8 +199,4 @@
             <cylinder radius="${wheel_radius-0.0001}" length="${wheel_width}"/>
           </geometry>
-			<!--<origin xyz="0.09002 1.1845 -0.8705" rpy="0 -0 0"/>
-			<geometry>
-				<mesh filename="package://m2020_urdf_models/rover/meshes/Wheel_LeftMiddle.dae" scale="1 1 1"/>
-			</geometry>-->
 		</collision>
 	</link>
@@ -229,5 +224,5 @@
 			<origin xyz="0 0 0" rpy="0 -0 0"/>
 			<mass value="${wheel_mass}"/>
-			<inertia ixx="${default_ixx}" ixy="0" ixz="0" iyy="${default_iyy}" iyz="0" izz="${default_izz}"/>
+			<inertia ixx="${wheel_ixx}" ixy="0" ixz="0" iyy="${wheel_iyy}" iyz="0" izz="${wheel_izz}"/>
 		</inertial>
 		<visual name="VisGeom_Wheel_LeftFront">
@@ -242,13 +237,9 @@
             <cylinder radius="${wheel_radius-0.0001}" length="${wheel_width}"/>
           </geometry>
-			<!--<origin xyz="-1.095 1.0625 -0.8705" rpy="0 -0 0"/>
-			<geometry>
-				<mesh filename="package://m2020_urdf_models/rover/meshes/Wheel_LeftFront.dae" scale="1 1 1"/>
-			</geometry>-->
 		</collision>
 	</link>
 	<link name="Body_RockerRight">
 		<inertial>
-			<origin xyz="-0.214 -0.79959 -0.2405" rpy="0 -0 0"/>
+			<origin xyz="0 0 0" rpy="0 0 0"/>
 			<mass value="${default_mass}"/>
 			<inertia ixx="${default_ixx}" ixy="0" ixz="0" iyy="${default_iyy}" iyz="0" izz="${default_izz}"/>
@@ -269,5 +260,5 @@
 	<link name="Body_BogieRight">
 		<inertial>
-			<origin xyz="0.54 -0.91959 -0.4705" rpy="0 -0 0"/>
+			<origin xyz="0 0 0" rpy="0 0 0"/>
 			<mass value="${default_mass}"/>
 			<inertia ixx="${default_ixx}" ixy="0" ixz="0" iyy="${default_iyy}" iyz="0" izz="${default_izz}"/>
@@ -288,5 +279,5 @@
 	<link name="Body_SteerRightRear">
 		<inertial>
-			<origin xyz="1.165 -1.0625 -0.8705" rpy="0 -0 0"/>
+			<origin xyz="0 0 0" rpy="0 0 0"/>
 			<mass value="${default_mass}"/>
 			<inertia ixx="${default_ixx}" ixy="0" ixz="0" iyy="${default_iyy}" iyz="0" izz="${default_izz}"/>
@@ -309,5 +300,5 @@
 			<origin xyz="0 0 0" rpy="0 -0 0"/>
 			<mass value="${wheel_mass}"/>
-			<inertia ixx="${default_ixx}" ixy="0" ixz="0" iyy="${default_iyy}" iyz="0" izz="${default_izz}"/>
+			<inertia ixx="${wheel_ixx}" ixy="0" ixz="0" iyy="${wheel_iyy}" iyz="0" izz="${wheel_izz}"/>
 		</inertial>
 		<visual name="VisGeom_Wheel_RightRear">
@@ -322,8 +313,4 @@
             <cylinder radius="${wheel_radius-0.0001}" length="${wheel_width}"/>
           </geometry>
-			<!--<origin xyz="1.165 -1.0625 -0.8705" rpy="0 -0 0"/>
-			<geometry>
-				<mesh filename="package://m2020_urdf_models/rover/meshes/Wheel_RightRear.dae" scale="1 1 1"/>
-			</geometry>-->
 		</collision>
 	</link>
@@ -332,5 +319,5 @@
 			<origin xyz="0 0 0" rpy="0 -0 0"/>
 			<mass value="${wheel_mass}"/>
-			<inertia ixx="${default_ixx}" ixy="0" ixz="0" iyy="${default_iyy}" iyz="0" izz="${default_izz}"/>
+			<inertia ixx="${wheel_ixx}" ixy="0" ixz="0" iyy="${wheel_iyy}" iyz="0" izz="${wheel_izz}"/>
 		</inertial>
 		<visual name="VisGeom_Wheel_RightMiddle">
@@ -345,13 +332,9 @@
             <cylinder radius="${wheel_radius-0.0001}" length="${wheel_width}"/>
           </geometry>
-		  <!--<origin xyz="0.09002 -1.1845 -0.8705" rpy="0 -0 0"/>
-			<geometry>
-				<mesh filename="package://m2020_urdf_models/rover/meshes/Wheel_RightMiddle.dae" scale="1 1 1"/>
-			</geometry>-->
 		</collision>
 	</link>
 	<link name="Body_SteerRightFront">
 		<inertial>
-			<origin xyz="-1.095 -1.0625 -0.8705" rpy="0 -0 0"/>
+			<origin xyz="0 0 0" rpy="0 -0 0"/>
 			<mass value="${default_mass}"/>
 			<inertia ixx="${default_ixx}" ixy="0" ixz="0" iyy="${default_iyy}" iyz="0" izz="${default_izz}"/>
@@ -374,5 +357,5 @@
 			<origin xyz="0 0 0" rpy="0 -0 0"/>
 			<mass value="${wheel_mass}"/>
-			<inertia ixx="${default_ixx}" ixy="0" ixz="0" iyy="${default_iyy}" iyz="0" izz="${default_izz}"/>
+			<inertia ixx="${wheel_ixx}" ixy="0" ixz="0" iyy="${wheel_iyy}" iyz="0" izz="${wheel_izz}"/>
 		</inertial>
 		<visual name="VisGeom_Wheel_RightFront">
@@ -387,8 +370,4 @@
             <cylinder radius="${wheel_radius-0.0001}" length="${wheel_width}"/>
           </geometry>
-			<!--<origin xyz="-1.095 -1.0625 -0.8705" rpy="0 -0 0"/>
-			<geometry>
-				<mesh filename="package://m2020_urdf_models/rover/meshes/Wheel_RightFront.dae" scale="1 1 1"/>
-			</geometry>-->
 		</collision>
 	</link>
@@ -433,5 +412,5 @@
 	<link name="Body_HGA_AZ">
 		<inertial>
-			<origin xyz="0.46 0.475 -0.0005" rpy="0 -0 0"/>
+			<origin xyz="0 0 0" rpy="0 0 0"/>
 			<mass value="${default_mass}"/>
 			<inertia ixx="${default_ixx}" ixy="0" ixz="0" iyy="${default_iyy}" iyz="0" izz="${default_izz}"/>
@@ -452,5 +431,5 @@
 	<link name="Body_HGA_EL">
 		<inertial>
-			<origin xyz="0.46 0.475 0.2475" rpy="0 -0 0"/>
+			<origin xyz="0 0 0" rpy="0 0 0"/>
 			<mass value="${default_mass}"/>
 			<inertia ixx="${default_ixx}" ixy="0" ixz="0" iyy="${default_iyy}" iyz="0" izz="${default_izz}"/>
@@ -471,5 +450,5 @@
 	<link name="Body_RA_Base">
 		<inertial>
-			<origin xyz="0 0 0" rpy="0 -0 0"/>
+			<origin xyz="0 0 0" rpy="0 0 0"/>
 			<mass value="${tiny_mass}"/>
 			<inertia ixx="${tiny_ixx}" ixy="0" ixz="0" iyy="${tiny_iyy}" iyz="0" izz="${tiny_izz}"/>
@@ -478,5 +457,5 @@
 	<link name="Body_RA_Link1">
 		<inertial>
-			<origin xyz="-1.1756 0.4515 -0.3116" rpy="0 -0 0"/>
+			<origin xyz="0 0 0" rpy="0 0 0"/>
 			<mass value="${default_mass}"/>
 			<inertia ixx="${default_ixx}" ixy="0" ixz="0" iyy="${default_iyy}" iyz="0" izz="${default_izz}"/>
@@ -516,5 +495,5 @@
 	<link name="Body_RA_Link3">
 		<inertial>
-			<origin xyz="0 0 0" rpy="0 -0 0"/>
+			<origin xyz="0 0 0" rpy="0 0 0"/>
 			<mass value="${default_mass}"/>
 			<inertia ixx="0.1" ixy="0" ixz="0" iyy="0.1" iyz="0" izz="0.1"/>
@@ -535,5 +514,5 @@
 	<link name="Body_RA_Link4">
 		<inertial>
-			<origin xyz="0 0 0" rpy="0 -0 0"/>
+			<origin xyz="0 0 0" rpy="0 0 0"/>
 			<mass value="${default_mass}"/>
 			<inertia ixx="${link4_ixx}" ixy="0" ixz="0" iyy="${link4_iyy}" iyz="0" izz="${link4_izz}"/>
@@ -629,5 +608,5 @@
 	<link name="Body_StabilizerFar">
 		<inertial>
-			<origin xyz="0 0 0" rpy="0 -0 0"/>
+			<origin xyz="0 0 0" rpy="0 0 0"/>
 			<mass value="${stabilizer_mass}"/>
 			<inertia ixx="${stabilizer_ixx}" ixy="0" ixz="0" iyy="${stabilizer_iyy}" iyz="0" izz="${stabilizer_izz}"/>
@@ -667,5 +646,5 @@
 	<link name="Body_WATSON_Cap">
 		<inertial>
-			<origin xyz="0 0 0" rpy="0 -0 0"/>
+			<origin xyz="0 0 0" rpy="0 0 0"/>
 			<mass value="${cap_mass}"/>
 			<inertia ixx="${cap_ixx}" ixy="0" ixz="0" iyy="${cap_iyy}" iyz="0" izz="${cap_izz}"/>
@@ -686,5 +665,5 @@
 	<link name="Body_SHERLOC_Cap">
 		<inertial>
-			<origin xyz="0 0 0" rpy="0 -0 0"/>
+			<origin xyz="0 0 0" rpy="0 0 0"/>
 			<mass value="${cap_mass}"/>
 			<inertia ixx="${cap_ixx}" ixy="0" ixz="0" iyy="${cap_iyy}" iyz="0" izz="${cap_izz}"/>
