Commit message: Added ns for gazebo

File: urdf/gazebo/kinect.gazebo.xacro (robot description, xacro)
@@ -1,5 +1,5 @@
 <?xml version="1.0"?>
 <robot xmlns:xacro="http://www.ros.org/wiki/xacro">
-<xacro:macro name="kinect_gazebo" params="prefix">
+<xacro:macro name="kinect_gazebo" params="prefix:='' robot_namespace:='' ">
   <gazebo reference="${prefix}kinect_link">
         <sensor type="depth" name="kinect_sensor">
@@ -24,5 +24,5 @@
                 <updateRate>0.0</updateRate>
                 <cameraName>kinect</cameraName>
-                <frameName>${prefix}kinect_optical_frame</frameName>
+                <frameName>${robot_namespace}/${prefix}kinect_optical_frame</frameName>
                 <imageTopicName>rgb/image_raw</imageTopicName>
                 <depthImageTopicName>depth/image_raw</depthImageTopicName>

File: urdf/gazebo/m2020.gazebo.components.xacro (robot description, xacro)
@@ -1,12 +1,14 @@
 <?xml version="1.0"?>
 <robot name="perseverance" xmlns:xacro="http://www.ros.org/wiki/xacro">
-  <xacro:include filename="$(find m2020_urdf_models)/urdf/gazebo/m2020.gazebo.component_macros.xacro" />
-  <xacro:include filename="$(find m2020_urdf_models)/urdf/gazebo/kinect.gazebo.xacro"/>
-  <xacro:include filename="$(find m2020_urdf_models)/urdf/gazebo/kinect.urdf.xacro"/>
-  <!-- build components -->
-  <xacro:m2020_base prefix="" />
-  <xacro:m2020_arm prefix=""/>
-  <xacro:m2020_head prefix=""/>
-  <xacro:kinect prefix="" parent="Frame_NCL_FOV"/>
-  <xacro:kinect_gazebo prefix=""/>
+  <xacro:macro name="m2020_gazebo_components"  params="robot_namespace:='' ">
+    <xacro:include filename="$(find m2020_urdf_models)/urdf/gazebo/m2020.gazebo.component_macros.xacro" />
+    <xacro:include filename="$(find m2020_urdf_models)/urdf/gazebo/kinect.gazebo.xacro"/>
+    <xacro:include filename="$(find m2020_urdf_models)/urdf/gazebo/kinect.urdf.xacro"/>
+    <!-- build components -->
+    <xacro:m2020_base prefix="" />
+    <xacro:m2020_arm prefix=""/>
+    <xacro:m2020_head prefix=""/>
+    <xacro:kinect prefix="" parent="Frame_NCL_FOV"/>
+    <xacro:kinect_gazebo prefix="" robot_namespace="${robot_namespace}"/>
+  </xacro:macro>
 </robot>

File: urdf/gazebo/m2020.gazebo.controllers.xacro (robot description, xacro)
@@ -1,12 +1,13 @@
 <?xml version="1.0"?>
 <robot xmlns:xacro="http://www.ros.org/wiki/xacro">
-  <xacro:arg name="robot_namespace" default="" />
-  <gazebo>
-    <plugin name="gazebo_ros_control" filename="libgazebo_ros_control.so">
-    <robotNamespace>$(arg robot_namespace)</robotNamespace>
-    <robotSimType>gazebo_ros_control/DefaultRobotHWSim</robotSimType>
-    <robotParam>robot_description</robotParam>
-    <legacyModeNS>true</legacyModeNS>
-  </plugin>
-  </gazebo>
+  <xacro:macro name="m2020_gazebo_ros_control"  params="robot_namespace:='' ">
+    <gazebo>
+      <plugin name="gazebo_ros_control" filename="libgazebo_ros_control.so">
+      <robotNamespace>${robot_namespace}</robotNamespace>
+      <robotSimType>gazebo_ros_control/DefaultRobotHWSim</robotSimType>
+      <robotParam>robot_description</robotParam>
+      <legacyModeNS>true</legacyModeNS>
+    </plugin>
+    </gazebo>
+  </xacro:macro>
 </robot>

File: urdf/m2020.sim.urdf.xacro (robot description, xacro)
@@ -1,5 +1,6 @@
 <?xml version="1.0" ?>
 <robot name="perseverance" xmlns:xacro="http://www.ros.org/wiki/xacro">
-  <xacro:property name="robot_name" value="perseverance" />
+  <xacro:arg name="robot_namespace" default="" />
+  <!--<xacro:property name="robot_name" value="perseverance" />-->
   <xacro:property name="mu1" value="100.0"/>
   <xacro:property name="mu2" value="100.0"/>
@@ -7,4 +8,6 @@
   <xacro:include filename="$(find m2020_urdf_models)/urdf/gazebo/m2020.gazebo.components.xacro" />
   <xacro:include filename="$(find m2020_urdf_models)/urdf/gazebo/m2020.gazebo.controllers.xacro" />
+  <xacro:m2020_gazebo_components robot_namespace="$(arg robot_namespace)"/>
+  <xacro:m2020_gazebo_ros_control robot_namespace="$(arg robot_namespace)"/>
   <!-- Parameters wheels -->
   <gazebo reference="LF_DRIVE">
