Commit message: reasonably working plugin for ingenuity in gazebo

File: urdf/gazebo/mhs.gazebo.component_macros.xacro (robot description, xacro)
@@ -64,8 +64,12 @@
     <xacro:gazebo_link prefix="${prefix}" link_name="Body_MHS_Leg03_v16" collide="true" static="${static}" gravity_off="${gravity_off}"/>
     <xacro:gazebo_link prefix="${prefix}" link_name="Body_MHS_Leg04_v16" collide="true" static="${static}" gravity_off="${gravity_off}"/>
+    <xacro:gazebo_joint prefix="${prefix}" joint_name="MHS_TopBlades_v16" kd="0" kp="1"/>
+    <xacro:gazebo_joint prefix="${prefix}" joint_name="MHS_BottomBlades_v16" kd="0" kp="1"/>
     <xacro:gazebo_joint prefix="${prefix}" joint_name="Joint_Leg01_Axis" kd="0" kp="1"/>
     <xacro:gazebo_joint prefix="${prefix}" joint_name="Joint_Leg02_Axis" kd="0" kp="1"/>
     <xacro:gazebo_joint prefix="${prefix}" joint_name="Joint_Leg03_Axis" kd="0" kp="1"/>
     <xacro:gazebo_joint prefix="${prefix}" joint_name="Joint_Leg04_Axis" kd="0" kp="1"/>
+    <xacro:gazebo_simple_trans prefix="${prefix}" joint_name="MHS_TopBlades_v16" reduction="1" tc="1"/>
+    <xacro:gazebo_simple_trans prefix="${prefix}" joint_name="MHS_BottomBlades_v16" reduction="1" tc="1"/>
     <xacro:gazebo_simple_trans prefix="${prefix}" joint_name="Joint_Leg01_Axis" reduction="1" tc="1"/>
     <xacro:gazebo_simple_trans prefix="${prefix}" joint_name="Joint_Leg02_Axis" reduction="1" tc="1"/>

File: urdf/mhs.urdf.xacro (robot description, xacro)
@@ -25,7 +25,7 @@
 		<collision name="ColGeom_MHS_MainBody_v16">
 			<origin xyz="0 0 0" rpy="0 -0 0"/>
-<!--       <geometry>
-        <box size="1.22 1.22 0.55" />
-      </geometry> -->
+      <!-- <geometry> -->
+        <!-- <box size="1.22 1.22 0.55" /> -->
+      <!-- </geometry> -->
 			<geometry>
 				<mesh filename="package://m2020_urdf_models/mhs/meshes/MHS_MainBody_v16.dae" scale="1 1 1"/>
