Commit message: some gain tuning

File: urdf/m2020.sim.urdf.xacro (robot description, xacro)
@@ -2,6 +2,6 @@
 <robot name="perseverance" xmlns:xacro="http://www.ros.org/wiki/xacro">
   <xacro:property name="robot_name" value="perseverance" />
-  <xacro:property name="mu1" value="100.0"/>
-  <xacro:property name="mu2" value="100.0"/>
+  <xacro:property name="mu1" value="100"/>
+  <xacro:property name="mu2" value="100"/>
   <xacro:include filename="$(find m2020_urdf_models)/urdf/m2020.traclabs.urdf.xacro" />
   <xacro:include filename="$(find m2020_urdf_models)/urdf/gazebo/m2020.gazebo.components.xacro" />
