Commit message: Works with dual perseverance

File: urdf/m2020.urdf.xacro (robot description, xacro)
@@ -24,4 +24,10 @@
 			</geometry>
 		</visual>
+		<collision name="CollGeom_CHASSIS">
+			<origin xyz="0.09002 0 -1.13338" rpy="0 -0 0"/>
+			<geometry>
+				<mesh filename="package://m2020_urdf_models/rover/meshes/CHASSIS.dae" scale="1 1 1"/>
+			</geometry>
+		</collision>
 	</link>
 	<link name="Body_MHS_DebrisShield">
@@ -104,4 +110,10 @@
 			</geometry>
 		</visual>
+		<collision name="ColGeom_Wheel_LeftRear">
+			<origin xyz="1.165 1.0625 -0.8705" rpy="0 -0 0"/>
+			<geometry>
+				<mesh filename="package://m2020_urdf_models/rover/meshes/Wheel_LeftRear.dae" scale="1 1 1"/>
+			</geometry>
+		</collision>
 	</link>
 	<link name="Body_WheelLeftMiddle">
@@ -117,4 +129,10 @@
 			</geometry>
 		</visual>
+		<collision name="ColGeom_Wheel_LeftMiddle">
+			<origin xyz="0.09002 1.1845 -0.8705" rpy="0 -0 0"/>
+			<geometry>
+				<mesh filename="package://m2020_urdf_models/rover/meshes/Wheel_LeftMiddle.dae" scale="1 1 1"/>
+			</geometry>
+		</collision>
 	</link>
 	<link name="Body_SteerLeftFront">
@@ -143,4 +161,10 @@
 			</geometry>
 		</visual>
+		<collision name="ColGeom_Wheel_LeftFront">
+			<origin xyz="-1.095 1.0625 -0.8705" rpy="0 -0 0"/>
+			<geometry>
+				<mesh filename="package://m2020_urdf_models/rover/meshes/Wheel_LeftFront.dae" scale="1 1 1"/>
+			</geometry>
+		</collision>
 	</link>
 	<link name="Body_RockerRight">
@@ -156,4 +180,10 @@
 			</geometry>
 		</visual>
+		<collision name="ColGeom_Right_Rocker">
+			<origin xyz="-0.214 -0.79959 -0.2405" rpy="0 -0 0"/>
+			<geometry>
+				<mesh filename="package://m2020_urdf_models/rover/meshes/Right_Rocker.dae" scale="1 1 1"/>
+			</geometry>
+		</collision>
 	</link>
 	<link name="Body_BogieRight">
@@ -169,4 +199,10 @@
 			</geometry>
 		</visual>
+		<collision name="ColGeom_Right_Bogie">
+			<origin xyz="0.54 -0.91959 -0.4705" rpy="0 -0 0"/>
+			<geometry>
+				<mesh filename="package://m2020_urdf_models/rover/meshes/Right_Bogie.dae" scale="1 1 1"/>
+			</geometry>
+		</collision>
 	</link>
 	<link name="Body_SteerRightRear">
@@ -195,4 +231,10 @@
 			</geometry>
 		</visual>
+		<collision name="ColGeom_Wheel_RightRear">
+			<origin xyz="1.165 -1.0625 -0.8705" rpy="0 -0 0"/>
+			<geometry>
+				<mesh filename="package://m2020_urdf_models/rover/meshes/Wheel_RightRear.dae" scale="1 1 1"/>
+			</geometry>
+		</collision>
 	</link>
 	<link name="Body_WheelRightMiddle">
@@ -208,4 +250,10 @@
 			</geometry>
 		</visual>
+		<collision name="ColGeom_Wheel_RightMiddle">
+			<origin xyz="0.09002 -1.1845 -0.8705" rpy="0 -0 0"/>
+			<geometry>
+				<mesh filename="package://m2020_urdf_models/rover/meshes/Wheel_RightMiddle.dae" scale="1 1 1"/>
+			</geometry>
+		</collision>
 	</link>
 	<link name="Body_SteerRightFront">
@@ -234,4 +282,10 @@
 			</geometry>
 		</visual>
+		<collision name="ColGeom_Wheel_RightFront">
+			<origin xyz="-1.095 -1.0625 -0.8705" rpy="0 -0 0"/>
+			<geometry>
+				<mesh filename="package://m2020_urdf_models/rover/meshes/Wheel_RightFront.dae" scale="1 1 1"/>
+			</geometry>
+		</collision>
 	</link>
 	<link name="Body_RSM_AZ">
@@ -306,4 +360,10 @@
 			</geometry>
 		</visual>
+		<collision name="ColGeom_Arm_LINK_1">
+			<origin xyz="-1.1756 0.4515 -0.3116" rpy="0 -0 0"/>
+			<geometry>
+				<mesh filename="package://m2020_urdf_models/rover/meshes/Arm_LINK_1.dae" scale="1 1 1"/>
+			</geometry>
+		</collision>
 	</link>
 	<link name="Body_RA_Link2">
@@ -319,4 +379,10 @@
 			</geometry>
 		</visual>
+		<collision name="ColGeom_Arm_LINK_2">
+			<origin xyz="-1.3416 0.4515 -0.3116" rpy="0 -0 0"/>
+			<geometry>
+				<mesh filename="package://m2020_urdf_models/rover/meshes/Arm_LINK_2.dae" scale="1 1 1"/>
+			</geometry>
+		</collision>
 	</link>
 	<link name="Body_RA_Link3">
@@ -332,4 +398,10 @@
 			</geometry>
 		</visual>
+		<collision name="ColGeom_Arm_LINK_3">
+			<origin xyz="-2.161 0.4515 -0.3116" rpy="0 -0 0"/>
+			<geometry>
+				<mesh filename="package://m2020_urdf_models/rover/meshes/Arm_LINK_3.dae" scale="1 1 1"/>
+			</geometry>
+		</collision>
 	</link>
 	<link name="Body_RA_Link4">
@@ -345,4 +417,10 @@
 			</geometry>
 		</visual>
+		<collision name="ColGeom_Arm_LINK_4">
+			<origin xyz="-2.9143 0.4515 -0.3116" rpy="0 -0 0"/>
+			<geometry>
+				<mesh filename="package://m2020_urdf_models/rover/meshes/Arm_LINK_4.dae" scale="1 1 1"/>
+			</geometry>
+		</collision>
 	</link>
 	<link name="Body_RA_Link5">
@@ -358,4 +436,10 @@
 			</geometry>
 		</visual>
+		<collision name="CollGeom_Arm_LINK_5">
+			<origin xyz="-2.7386 0.2724 -0.3116" rpy="0 -0 0"/>
+			<geometry>
+				<mesh filename="package://m2020_urdf_models/rover/meshes/Arm_LINK_5.dae" scale="1 1 1"/>
+			</geometry>
+		</collision>
 	</link>
 	<link name="Body_Turret">
@@ -371,4 +455,10 @@
 			</geometry>
 		</visual>
+		<collision name="ColGeom_Turret">
+			<origin xyz="0 0 0" rpy="0 -0 0"/>
+			<geometry>
+				<mesh filename="package://m2020_urdf_models/rover/meshes/Turret.dae" scale="1 1 1"/>
+			</geometry>
+		</collision>
 	</link>
 	<link name="Body_CorerFeed">

Commit message: Added head states

File: urdf/m2020.urdf.xacro (robot description, xacro)
@@ -4,4 +4,5 @@
 <robot name="perseverance" xmlns:xacro="http://www.ros.org/wiki/xacro">
   <xacro:property name="arm_joint_vel" value="0.2" /> <!-- original value: 1.79769e+308 -->
+  <xacro:property name="head_joint_vel" value="1.0" /> <!-- original value: 1.79769e+308 -->
 	<!--<link name="ground">
 		<inertial>
@@ -1244,5 +1245,5 @@
 		<child link="Body_RSM_AZ"/>
 		<axis xyz="0 0 1"/>
-		<limit lower="0" upper="6.31809" effort="1.79769e+308" velocity="1.79769e+308"/>
+		<limit lower="0" upper="6.31809" effort="1.79769e+308" velocity="${head_joint_vel}"/>
 	</joint>
 	<joint name="RSM_EL_ENC" type="revolute">
@@ -1251,5 +1252,5 @@
 		<child link="Body_RSM_EL"/>
 		<axis xyz="0 1 0"/>
-		<limit lower="0" upper="3.1765" effort="1.79769e+308" velocity="1.79769e+308"/>
+		<limit lower="0" upper="3.1765" effort="1.79769e+308" velocity="${head_joint_vel}"/>
 	</joint>
 	<joint name="HGA_AZ" type="revolute">

Commit message: Added filter

File: urdf/m2020.urdf.xacro (robot description, xacro)
@@ -552,571 +552,85 @@
 		</visual>
 	</link>
-	<link name="Frame_RNAV">
-		<inertial>
-			<origin xyz="0 0 0" rpy="0 -0 0"/>
-			<mass value="0"/>
-			<inertia ixx="0" ixy="0" ixz="0" iyy="0" iyz="0" izz="0"/>
-		</inertial>
-	</link>
-	<link name="Frame_RMECH">
-		<inertial>
-			<origin xyz="0 0 0" rpy="0 -0 0"/>
-			<mass value="0"/>
-			<inertia ixx="0" ixy="0" ixz="0" iyy="0" iyz="0" izz="0"/>
-		</inertial>
-	</link>
-	<link name="Frame_FHCB">
-		<inertial>
-			<origin xyz="0 0 0" rpy="0 -0 0"/>
-			<mass value="0"/>
-			<inertia ixx="0" ixy="0" ixz="0" iyy="0" iyz="0" izz="0"/>
-		</inertial>
-	</link>
-	<link name="Frame_FHC1">
-		<inertial>
-			<origin xyz="0 0 0" rpy="0 -0 0"/>
-			<mass value="0"/>
-			<inertia ixx="0" ixy="0" ixz="0" iyy="0" iyz="0" izz="0"/>
-		</inertial>
-	</link>
-	<link name="Frame_FHC2">
-		<inertial>
-			<origin xyz="0 0 0" rpy="0 -0 0"/>
-			<mass value="0"/>
-			<inertia ixx="0" ixy="0" ixz="0" iyy="0" iyz="0" izz="0"/>
-		</inertial>
-	</link>
-	<link name="Frame_FHC3">
-		<inertial>
-			<origin xyz="0 0 0" rpy="0 -0 0"/>
-			<mass value="0"/>
-			<inertia ixx="0" ixy="0" ixz="0" iyy="0" iyz="0" izz="0"/>
-		</inertial>
-	</link>
-	<link name="Frame_FHC4">
-		<inertial>
-			<origin xyz="0 0 0" rpy="0 -0 0"/>
-			<mass value="0"/>
-			<inertia ixx="0" ixy="0" ixz="0" iyy="0" iyz="0" izz="0"/>
-		</inertial>
-	</link>
-	<link name="Frame_FHC1_FOV">
-		<inertial>
-			<origin xyz="0 0 0" rpy="0 -0 0"/>
-			<mass value="0"/>
-			<inertia ixx="0" ixy="0" ixz="0" iyy="0" iyz="0" izz="0"/>
-		</inertial>
-	</link>
-	<link name="Frame_FHC2_FOV">
-		<inertial>
-			<origin xyz="0 0 0" rpy="0 -0 0"/>
-			<mass value="0"/>
-			<inertia ixx="0" ixy="0" ixz="0" iyy="0" iyz="0" izz="0"/>
-		</inertial>
-	</link>
-	<link name="Frame_FHC3_FOV">
-		<inertial>
-			<origin xyz="0 0 0" rpy="0 -0 0"/>
-			<mass value="0"/>
-			<inertia ixx="0" ixy="0" ixz="0" iyy="0" iyz="0" izz="0"/>
-		</inertial>
-	</link>
-	<link name="Frame_FHC4_FOV">
-		<inertial>
-			<origin xyz="0 0 0" rpy="0 -0 0"/>
-			<mass value="0"/>
-			<inertia ixx="0" ixy="0" ixz="0" iyy="0" iyz="0" izz="0"/>
-		</inertial>
-	</link>
-	<link name="Frame_RHC1">
-		<inertial>
-			<origin xyz="0 0 0" rpy="0 -0 0"/>
-			<mass value="0"/>
-			<inertia ixx="0" ixy="0" ixz="0" iyy="0" iyz="0" izz="0"/>
-		</inertial>
-	</link>
-	<link name="Frame_RHC2">
-		<inertial>
-			<origin xyz="0 0 0" rpy="0 -0 0"/>
-			<mass value="0"/>
-			<inertia ixx="0" ixy="0" ixz="0" iyy="0" iyz="0" izz="0"/>
-		</inertial>
-	</link>
-	<link name="Frame_RHC1_FOV">
-		<inertial>
-			<origin xyz="0 0 0" rpy="0 -0 0"/>
-			<mass value="0"/>
-			<inertia ixx="0" ixy="0" ixz="0" iyy="0" iyz="0" izz="0"/>
-		</inertial>
-	</link>
-	<link name="Frame_RHC2_FOV">
-		<inertial>
-			<origin xyz="0 0 0" rpy="0 -0 0"/>
-			<mass value="0"/>
-			<inertia ixx="0" ixy="0" ixz="0" iyy="0" iyz="0" izz="0"/>
-		</inertial>
-	</link>
-	<link name="Frame_ATS1">
-		<inertial>
-			<origin xyz="0 0 0" rpy="0 -0 0"/>
-			<mass value="0"/>
-			<inertia ixx="0" ixy="0" ixz="0" iyy="0" iyz="0" izz="0"/>
-		</inertial>
-	</link>
-	<link name="Frame_ATS2">
-		<inertial>
-			<origin xyz="0 0 0" rpy="0 -0 0"/>
-			<mass value="0"/>
-			<inertia ixx="0" ixy="0" ixz="0" iyy="0" iyz="0" izz="0"/>
-		</inertial>
-	</link>
-	<link name="Frame_ATS3">
-		<inertial>
-			<origin xyz="0 0 0" rpy="0 -0 0"/>
-			<mass value="0"/>
-			<inertia ixx="0" ixy="0" ixz="0" iyy="0" iyz="0" izz="0"/>
-		</inertial>
-	</link>
-	<link name="Frame_ATS4">
-		<inertial>
-			<origin xyz="0 0 0" rpy="0 -0 0"/>
-			<mass value="0"/>
-			<inertia ixx="0" ixy="0" ixz="0" iyy="0" iyz="0" izz="0"/>
-		</inertial>
-	</link>
-	<link name="Frame_ATS5">
-		<inertial>
-			<origin xyz="0 0 0" rpy="0 -0 0"/>
-			<mass value="0"/>
-			<inertia ixx="0" ixy="0" ixz="0" iyy="0" iyz="0" izz="0"/>
-		</inertial>
-	</link>
-	<link name="Frame_HS">
-		<inertial>
-			<origin xyz="0 0 0" rpy="0 -0 0"/>
-			<mass value="0"/>
-			<inertia ixx="0" ixy="0" ixz="0" iyy="0" iyz="0" izz="0"/>
-		</inertial>
-	</link>
-	<link name="Frame_ICU">
-		<inertial>
-			<origin xyz="0 0 0" rpy="0 -0 0"/>
-			<mass value="0"/>
-			<inertia ixx="0" ixy="0" ixz="0" iyy="0" iyz="0" izz="0"/>
-		</inertial>
-	</link>
-	<link name="Frame_RDS">
-		<inertial>
-			<origin xyz="0 0 0" rpy="0 -0 0"/>
-			<mass value="0"/>
-			<inertia ixx="0" ixy="0" ixz="0" iyy="0" iyz="0" izz="0"/>
-		</inertial>
-	</link>
-	<link name="Frame_TIRS">
-		<inertial>
-			<origin xyz="0 0 0" rpy="0 -0 0"/>
-			<mass value="0"/>
-			<inertia ixx="0" ixy="0" ixz="0" iyy="0" iyz="0" izz="0"/>
-		</inertial>
-	</link>
-	<link name="Frame_WS1">
-		<inertial>
-			<origin xyz="0 0 0" rpy="0 -0 0"/>
-			<mass value="0"/>
-			<inertia ixx="0" ixy="0" ixz="0" iyy="0" iyz="0" izz="0"/>
-		</inertial>
-	</link>
-	<link name="Frame_WS2">
-		<inertial>
-			<origin xyz="0 0 0" rpy="0 -0 0"/>
-			<mass value="0"/>
-			<inertia ixx="0" ixy="0" ixz="0" iyy="0" iyz="0" izz="0"/>
-		</inertial>
-	</link>
-	<link name="Frame_MOXIE">
-		<inertial>
-			<origin xyz="0 0 0" rpy="0 -0 0"/>
-			<mass value="0"/>
-			<inertia ixx="0" ixy="0" ixz="0" iyy="0" iyz="0" izz="0"/>
-		</inertial>
-	</link>
-	<link name="Frame_MI">
-		<inertial>
-			<origin xyz="0 0 0" rpy="0 -0 0"/>
-			<mass value="0"/>
-			<inertia ixx="0" ixy="0" ixz="0" iyy="0" iyz="0" izz="0"/>
-		</inertial>
-	</link>
-	<link name="Frame_MAZ">
-		<inertial>
-			<origin xyz="0 0 0" rpy="0 -0 0"/>
-			<mass value="0"/>
-			<inertia ixx="0" ixy="0" ixz="0" iyy="0" iyz="0" izz="0"/>
-		</inertial>
-	</link>
-	<link name="Frame_MEL">
-		<inertial>
-			<origin xyz="0 0 0" rpy="0 -0 0"/>
-			<mass value="0"/>
-			<inertia ixx="0" ixy="0" ixz="0" iyy="0" iyz="0" izz="0"/>
-		</inertial>
-	</link>
-	<link name="Frame_SCI">
-		<inertial>
-			<origin xyz="0 0 0" rpy="0 -0 0"/>
-			<mass value="0"/>
-			<inertia ixx="0" ixy="0" ixz="0" iyy="0" iyz="0" izz="0"/>
-		</inertial>
-	</link>
-	<link name="Frame_SCRMI">
-		<inertial>
-			<origin xyz="0 0 0" rpy="0 -0 0"/>
-			<mass value="0"/>
-			<inertia ixx="0" ixy="0" ixz="0" iyy="0" iyz="0" izz="0"/>
-		</inertial>
-	</link>
-	<link name="Frame_SCLIBS">
-		<inertial>
-			<origin xyz="0 0 0" rpy="0 -0 0"/>
-			<mass value="0"/>
-			<inertia ixx="0" ixy="0" ixz="0" iyy="0" iyz="0" izz="0"/>
-		</inertial>
-	</link>
-	<link name="Frame_SCIR">
-		<inertial>
-			<origin xyz="0 0 0" rpy="0 -0 0"/>
-			<mass value="0"/>
-			<inertia ixx="0" ixy="0" ixz="0" iyy="0" iyz="0" izz="0"/>
-		</inertial>
-	</link>
-	<link name="Frame_MCL">
-		<inertial>
-			<origin xyz="0 0 0" rpy="0 -0 0"/>
-			<mass value="0"/>
-			<inertia ixx="0" ixy="0" ixz="0" iyy="0" iyz="0" izz="0"/>
-		</inertial>
-	</link>
-	<link name="Frame_MCR">
-		<inertial>
-			<origin xyz="0 0 0" rpy="0 -0 0"/>
-			<mass value="0"/>
-			<inertia ixx="0" ixy="0" ixz="0" iyy="0" iyz="0" izz="0"/>
-		</inertial>
-	</link>
-	<link name="Frame_NCL">
-		<inertial>
-			<origin xyz="0 0 0" rpy="0 -0 0"/>
-			<mass value="0"/>
-			<inertia ixx="0" ixy="0" ixz="0" iyy="0" iyz="0" izz="0"/>
-		</inertial>
-	</link>
-	<link name="Frame_NCR">
-		<inertial>
-			<origin xyz="0 0 0" rpy="0 -0 0"/>
-			<mass value="0"/>
-			<inertia ixx="0" ixy="0" ixz="0" iyy="0" iyz="0" izz="0"/>
-		</inertial>
-	</link>
-	<link name="Frame_NCL_FOV">
-		<inertial>
-			<origin xyz="0 0 0" rpy="0 -0 0"/>
-			<mass value="0"/>
-			<inertia ixx="0" ixy="0" ixz="0" iyy="0" iyz="0" izz="0"/>
-		</inertial>
-	</link>
-	<link name="Frame_NCR_FOV">
-		<inertial>
-			<origin xyz="0 0 0" rpy="0 -0 0"/>
-			<mass value="0"/>
-			<inertia ixx="0" ixy="0" ixz="0" iyy="0" iyz="0" izz="0"/>
-		</inertial>
-	</link>
-	<link name="Frame_ROCKER_L">
-		<inertial>
-			<origin xyz="0 0 0" rpy="0 -0 0"/>
-			<mass value="0"/>
-			<inertia ixx="0" ixy="0" ixz="0" iyy="0" iyz="0" izz="0"/>
-		</inertial>
-	</link>
-	<link name="Frame_ROCKER_R">
-		<inertial>
-			<origin xyz="0 0 0" rpy="0 -0 0"/>
-			<mass value="0"/>
-			<inertia ixx="0" ixy="0" ixz="0" iyy="0" iyz="0" izz="0"/>
-		</inertial>
-	</link>
-	<link name="Frame_BOGIE_L">
-		<inertial>
-			<origin xyz="0 0 0" rpy="0 -0 0"/>
-			<mass value="0"/>
-			<inertia ixx="0" ixy="0" ixz="0" iyy="0" iyz="0" izz="0"/>
-		</inertial>
-	</link>
-	<link name="Frame_BOGIE_R">
-		<inertial>
-			<origin xyz="0 0 0" rpy="0 -0 0"/>
-			<mass value="0"/>
-			<inertia ixx="0" ixy="0" ixz="0" iyy="0" iyz="0" izz="0"/>
-		</inertial>
-	</link>
-	<link name="Frame_DIFF">
-		<inertial>
-			<origin xyz="0 0 0" rpy="0 -0 0"/>
-			<mass value="0"/>
-			<inertia ixx="0" ixy="0" ixz="0" iyy="0" iyz="0" izz="0"/>
-		</inertial>
-	</link>
-	<link name="Frame_STEER_LF">
-		<inertial>
-			<origin xyz="0 0 0" rpy="0 -0 0"/>
-			<mass value="0"/>
-			<inertia ixx="0" ixy="0" ixz="0" iyy="0" iyz="0" izz="0"/>
-		</inertial>
-	</link>
-	<link name="Frame_STEER_LR">
-		<inertial>
-			<origin xyz="0 0 0" rpy="0 -0 0"/>
-			<mass value="0"/>
-			<inertia ixx="0" ixy="0" ixz="0" iyy="0" iyz="0" izz="0"/>
-		</inertial>
-	</link>
-	<link name="Frame_STEER_RF">
-		<inertial>
-			<origin xyz="0 0 0" rpy="0 -0 0"/>
-			<mass value="0"/>
-			<inertia ixx="0" ixy="0" ixz="0" iyy="0" iyz="0" izz="0"/>
-		</inertial>
-	</link>
-	<link name="Frame_STEER_RR">
-		<inertial>
-			<origin xyz="0 0 0" rpy="0 -0 0"/>
-			<mass value="0"/>
-			<inertia ixx="0" ixy="0" ixz="0" iyy="0" iyz="0" izz="0"/>
-		</inertial>
-	</link>
-	<link name="Frame_WHEEL_LF">
-		<inertial>
-			<origin xyz="0 0 0" rpy="0 -0 0"/>
-			<mass value="0"/>
-			<inertia ixx="0" ixy="0" ixz="0" iyy="0" iyz="0" izz="0"/>
-		</inertial>
-	</link>
-	<link name="Frame_WHEEL_LM">
-		<inertial>
-			<origin xyz="0 0 0" rpy="0 -0 0"/>
-			<mass value="0"/>
-			<inertia ixx="0" ixy="0" ixz="0" iyy="0" iyz="0" izz="0"/>
-		</inertial>
-	</link>
-	<link name="Frame_WHEEL_LR">
-		<inertial>
-			<origin xyz="0 0 0" rpy="0 -0 0"/>
-			<mass value="0"/>
-			<inertia ixx="0" ixy="0" ixz="0" iyy="0" iyz="0" izz="0"/>
-		</inertial>
-	</link>
-	<link name="Frame_WHEEL_RF">
-		<inertial>
-			<origin xyz="0 0 0" rpy="0 -0 0"/>
-			<mass value="0"/>
-			<inertia ixx="0" ixy="0" ixz="0" iyy="0" iyz="0" izz="0"/>
-		</inertial>
-	</link>
-	<link name="Frame_WHEEL_RM">
-		<inertial>
-			<origin xyz="0 0 0" rpy="0 -0 0"/>
-			<mass value="0"/>
-			<inertia ixx="0" ixy="0" ixz="0" iyy="0" iyz="0" izz="0"/>
-		</inertial>
-	</link>
-	<link name="Frame_WHEEL_RR">
-		<inertial>
-			<origin xyz="0 0 0" rpy="0 -0 0"/>
-			<mass value="0"/>
-			<inertia ixx="0" ixy="0" ixz="0" iyy="0" iyz="0" izz="0"/>
-		</inertial>
-	</link>
-	<link name="Frame_RIMUA">
-		<inertial>
-			<origin xyz="0 0 0" rpy="0 -0 0"/>
-			<mass value="0"/>
-			<inertia ixx="0" ixy="0" ixz="0" iyy="0" iyz="0" izz="0"/>
-		</inertial>
-	</link>
-	<link name="Frame_RIMUB">
-		<inertial>
-			<origin xyz="0 0 0" rpy="0 -0 0"/>
-			<mass value="0"/>
-			<inertia ixx="0" ixy="0" ixz="0" iyy="0" iyz="0" izz="0"/>
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
Commit message: WYCLIFF -- THis will be a local branch

File: urdf/m2020.urdf.xacro (robot description, xacro)
@@ -22,5 +22,6 @@
 			<origin xyz="0.09002 0 -1.13338" rpy="0 -0 0"/>
 			<geometry>
-				<mesh filename="package://m2020_urdf_models/rover/meshes/CHASSIS.dae" scale="1 1 1"/>
+				<!--<mesh filename="package://m2020_urdf_models/rover/meshes/CHASSIS.dae" scale="1 1 1"/>-->
+				<mesh filename="package://m2020_urdf_models/rover/meshes/CHASSIS_low_res.stl" scale="1 1 1"/>
 			</geometry>
 		</visual>
@@ -28,5 +29,6 @@
 			<origin xyz="0.09002 0 -1.13338" rpy="0 -0 0"/>
 			<geometry>
-				<mesh filename="package://m2020_urdf_models/rover/meshes/CHASSIS.dae" scale="1 1 1"/>
+				<!--<mesh filename="package://m2020_urdf_models/rover/meshes/CHASSIS.dae" scale="1 1 1"/>-->
+				<mesh filename="package://m2020_urdf_models/rover/meshes/CHASSIS_low_res.stl" scale="1 1 1"/>
 			</geometry>
 		</collision>
@@ -56,5 +58,6 @@
 			<origin xyz="0.142 0 0" rpy="0 -0 0"/>
 			<geometry>
-				<mesh filename="package://m2020_urdf_models/rover/meshes/CenterDifferential.dae" scale="1 1 1"/>
+				<!-- <mesh filename="package://m2020_urdf_models/rover/meshes/CenterDifferential.dae" scale="1 1 1"/> -->
+				<mesh filename="package://m2020_urdf_models/rover/meshes/CenterDifferential_low_res.stl" scale="1 1 1"/>
 			</geometry>
 		</visual>
@@ -69,5 +72,6 @@
 			<origin xyz="-0.214 0.79959 -0.2405" rpy="0 -0 0"/>
 			<geometry>
-				<mesh filename="package://m2020_urdf_models/rover/meshes/Left_Rocker.dae" scale="1 1 1"/>
+				<!-- <mesh filename="package://m2020_urdf_models/rover/meshes/Left_Rocker.dae" scale="1 1 1"/> -->
+				<mesh filename="package://m2020_urdf_models/rover/meshes/Left_Rocker_low_res.stl" scale="1 1 1"/>
 			</geometry>
 		</visual>
@@ -82,5 +86,6 @@
 			<origin xyz="0.54 0.91959 -0.4705" rpy="0 -0 0"/>
 			<geometry>
-				<mesh filename="package://m2020_urdf_models/rover/meshes/Left_Bogie.dae" scale="1 1 1"/>
+				<!-- <mesh filename="package://m2020_urdf_models/rover/meshes/Left_Bogie.dae" scale="1 1 1"/> -->
+				<mesh filename="package://m2020_urdf_models/rover/meshes/Left_Bogie_low_res.stl" scale="1 1 1"/>
 			</geometry>
 		</visual>
@@ -197,5 +202,6 @@
 			<origin xyz="0.54 -0.91959 -0.4705" rpy="0 -0 0"/>
 			<geometry>
-				<mesh filename="package://m2020_urdf_models/rover/meshes/Right_Bogie.dae" scale="1 1 1"/>
+				<!-- <mesh filename="package://m2020_urdf_models/rover/meshes/Right_Bogie.dae" scale="1 1 1"/> -->
+				<mesh filename="package://m2020_urdf_models/rover/meshes/Right_Bogie_low_res.stl" scale="1 1 1"/>
 			</geometry>
 		</visual>
@@ -203,5 +209,6 @@
 			<origin xyz="0.54 -0.91959 -0.4705" rpy="0 -0 0"/>
 			<geometry>
-				<mesh filename="package://m2020_urdf_models/rover/meshes/Right_Bogie.dae" scale="1 1 1"/>
+				<!-- <mesh filename="package://m2020_urdf_models/rover/meshes/Right_Bogie.dae" scale="1 1 1"/> -->
+				<mesh filename="package://m2020_urdf_models/rover/meshes/Right_Bogie_low_res.stl" scale="1 1 1"/>
 			</geometry>
 		</collision>

Commit message: WYCLIFF -- Low res directory     in m2020-urdf-models/rover/meshes/low_res

File: urdf/m2020.urdf.xacro (robot description, xacro)
@@ -23,5 +23,5 @@
 			<geometry>
 				<!--<mesh filename="package://m2020_urdf_models/rover/meshes/CHASSIS.dae" scale="1 1 1"/>-->
-				<mesh filename="package://m2020_urdf_models/rover/meshes/CHASSIS_low_res.stl" scale="1 1 1"/>
+				<mesh filename="package://m2020_urdf_models/rover/meshes/low_res/CHASSIS_low_res.stl" scale="1 1 1"/>
 			</geometry>
 		</visual>
@@ -30,5 +30,5 @@
 			<geometry>
 				<!--<mesh filename="package://m2020_urdf_models/rover/meshes/CHASSIS.dae" scale="1 1 1"/>-->
-				<mesh filename="package://m2020_urdf_models/rover/meshes/CHASSIS_low_res.stl" scale="1 1 1"/>
+				<mesh filename="package://m2020_urdf_models/rover/meshes/low_res/CHASSIS_low_res.stl" scale="1 1 1"/>
 			</geometry>
 		</collision>
@@ -59,5 +59,5 @@
 			<geometry>
 				<!-- <mesh filename="package://m2020_urdf_models/rover/meshes/CenterDifferential.dae" scale="1 1 1"/> -->
-				<mesh filename="package://m2020_urdf_models/rover/meshes/CenterDifferential_low_res.stl" scale="1 1 1"/>
+				<mesh filename="package://m2020_urdf_models/rover/meshes/low_res/CenterDifferential_low_res.stl" scale="1 1 1"/>
 			</geometry>
 		</visual>
@@ -73,5 +73,5 @@
 			<geometry>
 				<!-- <mesh filename="package://m2020_urdf_models/rover/meshes/Left_Rocker.dae" scale="1 1 1"/> -->
-				<mesh filename="package://m2020_urdf_models/rover/meshes/Left_Rocker_low_res.stl" scale="1 1 1"/>
+				<mesh filename="package://m2020_urdf_models/rover/meshes/low_res/Left_Rocker_low_res.stl" scale="1 1 1"/>
 			</geometry>
 		</visual>
@@ -87,5 +87,5 @@
 			<geometry>
 				<!-- <mesh filename="package://m2020_urdf_models/rover/meshes/Left_Bogie.dae" scale="1 1 1"/> -->
-				<mesh filename="package://m2020_urdf_models/rover/meshes/Left_Bogie_low_res.stl" scale="1 1 1"/>
+				<mesh filename="package://m2020_urdf_models/rover/meshes/low_res/Left_Bogie_low_res.stl" scale="1 1 1"/>
 			</geometry>
 		</visual>
@@ -203,5 +203,5 @@
 			<geometry>
 				<!-- <mesh filename="package://m2020_urdf_models/rover/meshes/Right_Bogie.dae" scale="1 1 1"/> -->
-				<mesh filename="package://m2020_urdf_models/rover/meshes/Right_Bogie_low_res.stl" scale="1 1 1"/>
+				<mesh filename="package://m2020_urdf_models/rover/meshes/low_res/Right_Bogie_low_res.stl" scale="1 1 1"/>
 			</geometry>
 		</visual>
@@ -210,5 +210,5 @@
 			<geometry>
 				<!-- <mesh filename="package://m2020_urdf_models/rover/meshes/Right_Bogie.dae" scale="1 1 1"/> -->
-				<mesh filename="package://m2020_urdf_models/rover/meshes/Right_Bogie_low_res.stl" scale="1 1 1"/>
+				<mesh filename="package://m2020_urdf_models/rover/meshes/low_res/Right_Bogie_low_res.stl" scale="1 1 1"/>
 			</geometry>
 		</collision>
