Commit message: Improving gazebo sim

File: urdf/m2020.traclabs.urdf.xacro (robot description, xacro)
@@ -3,10 +3,43 @@
 <!-- m2020.gazebo.urdf.xacro: File that was vastly modified by TRACLabs to work with Gazebo -->
 <robot name="perseverance" xmlns:xacro="http://www.ros.org/wiki/xacro">
+  <!-- TRACLABS NOTES CONVERSION: Commented out: 	<link name="Body_CorerFeed"> CHECK OUT LATER!  -->
+  <xacro:include filename="$(find m2020_urdf_models)/urdf/gazebo/m2020.gazebo.component_macros.xacro"/>
   <xacro:property name="arm_joint_vel" value="0.2" /> <!-- original value: 1.79769e+308 -->
   <xacro:property name="head_joint_vel" value="1.0" /> <!-- original value: 1.79769e+308 -->
-  <xacro:property name="default_mass" value="1.0" />
+  <xacro:property name="arm_default_effort" value="100.0" /> <!-- original value: 1.79769e+308 -->
+  <xacro:property name="stabilizer_default_vel" value="0.5"/> <!-- original value: 1.79769e+308 -->
+  <xacro:property name="stabilizer_default_effort" value="50"/> <!-- original value: 1.79769e+308 -->
+  <xacro:property name="arm_default_damping" value="1.0"/>
+  <xacro:property name="arm_default_friction" value="10.0"/>
+  <xacro:property name="default_mass" value="3.0" />
   <xacro:property name="default_ixx" value="0.2" />
   <xacro:property name="default_iyy" value="0.2" />
   <xacro:property name="default_izz" value="0.2" />
+  <xacro:property name="link4_ixx" value="0.05" />
+  <xacro:property name="link4_iyy" value="0.05" />
+  <xacro:property name="link4_izz" value="0.05" />
+  <xacro:property name="link5_ixx" value="0.05" />
+  <xacro:property name="link5_iyy" value="0.05" />
+  <xacro:property name="link5_izz" value="0.05" />
+  <xacro:property name="stabilizer_mass" value="0.5"/>
+  <xacro:property name="stabilizer_ixx" value="0.01" />
+  <xacro:property name="stabilizer_iyy" value="0.01" />
+  <xacro:property name="stabilizer_izz" value="0.01" />
+  <xacro:property name="cap_mass" value="0.1"/>
+  <xacro:property name="cap_ixx" value="0.005" />
+  <xacro:property name="cap_iyy" value="0.005" />
+  <xacro:property name="cap_izz" value="0.005" />
+  <xacro:property name="turret_mass" value="1.0"/>
+  <xacro:property name="turret_ixx" value="0.1" />
+  <xacro:property name="turret_iyy" value="0.1" />
+  <xacro:property name="turret_izz" value="0.1" />
+  <!-- For link with no visual, no collision, just a frame -->
+  <xacro:property name="tiny_mass" value="0.001"/>
+  <xacro:property name="tiny_ixx" value="0.00001" />
+  <xacro:property name="tiny_iyy" value="0.00001" />
+  <xacro:property name="tiny_izz" value="0.00001" />
+  <xacro:property name="head_damping" value="1.0"/>
+  <xacro:property name="head_friction" value="10.0"/>
+  <xacro:property name="head_effort" value="100.0" />
 	<link name="base_footprint"/>
 	<link name="Body_Chassis">
@@ -331,5 +364,5 @@
 	<link name="Body_RSM_AZ">
 		<inertial>
-			<origin xyz="-0.714017 -0.559028 0.78589" rpy="0 -0 0"/>
+			<origin xyz="0 0 0" rpy="0 -0 0"/>
 			<mass value="${default_mass}"/>
 			<inertia ixx="${default_ixx}" ixy="0" ixz="0" iyy="${default_iyy}" iyz="0" izz="${default_izz}"/>
@@ -350,5 +383,5 @@
 	<link name="Body_RSM_EL">
 		<inertial>
-			<origin xyz="-0.714017 -0.559028 0.78589" rpy="0 -0 0"/>
+			<origin xyz="0 0 0" rpy="0 -0 0"/>
 			<mass value="${default_mass}"/>
 			<inertia ixx="${default_ixx}" ixy="0" ixz="0" iyy="${default_iyy}" iyz="0" izz="${default_izz}"/>
@@ -406,9 +439,9 @@
 	</link>
 	<link name="Body_RA_Base">
-		<!--<inertial>
+		<inertial>
 			<origin xyz="0 0 0" rpy="0 -0 0"/>
-			<mass value="${default_mass}"/>
-			<inertia ixx="${default_ixx}" ixy="0" ixz="0" iyy="${default_iyy}" iyz="0" izz="${default_izz}"/>
-		</inertial>--> <!-- Commented out TRACLabs-->
+			<mass value="${tiny_mass}"/>
+			<inertia ixx="${tiny_ixx}" ixy="0" ixz="0" iyy="${tiny_iyy}" iyz="0" izz="${tiny_izz}"/>
+		</inertial>
 	</link>
 	<link name="Body_RA_Link1">
@@ -433,5 +466,5 @@
 	<link name="Body_RA_Link2">
 		<inertial>
-			<origin xyz="-1.3416 0.4515 -0.3116" rpy="0 -0 0"/>
+			<origin xyz="0 0 0" rpy="0 -0 0"/>
 			<mass value="${default_mass}"/>
 			<inertia ixx="${default_ixx}" ixy="0" ixz="0" iyy="${default_iyy}" iyz="0" izz="${default_izz}"/>
@@ -452,7 +485,7 @@
 	<link name="Body_RA_Link3">
 		<inertial>
-			<origin xyz="-2.161 0.4515 -0.3116" rpy="0 -0 0"/>
-			<mass value="${default_mass}"/>
-			<inertia ixx="${default_ixx}" ixy="0" ixz="0" iyy="${default_iyy}" iyz="0" izz="${default_izz}"/>
+			<origin xyz="0 0 0" rpy="0 -0 0"/>
+			<mass value="${default_mass}"/>
+			<inertia ixx="0.1" ixy="0" ixz="0" iyy="0.1" iyz="0" izz="0.1"/>
 		</inertial>
 		<visual name="VisGeom_Arm_LINK_3">
@@ -471,7 +504,7 @@
 	<link name="Body_RA_Link4">
 		<inertial>
-			<origin xyz="-2.9143 0.4515 -0.3116" rpy="0 -0 0"/>
-			<mass value="${default_mass}"/>
-			<inertia ixx="${default_ixx}" ixy="0" ixz="0" iyy="${default_iyy}" iyz="0" izz="${default_izz}"/>
+			<origin xyz="0 0 0" rpy="0 -0 0"/>
+			<mass value="${default_mass}"/>
+			<inertia ixx="${link4_ixx}" ixy="0" ixz="0" iyy="${link4_iyy}" iyz="0" izz="${link4_izz}"/>
 		</inertial>
 		<visual name="VisGeom_Arm_LINK_4">
@@ -489,8 +522,8 @@
 	</link>
 	<link name="Body_RA_Link5">
-		<inertial>
-			<origin xyz="-2.7386 0.2724 -0.3116" rpy="0 -0 0"/>
-			<mass value="${default_mass}"/>
-			<inertia ixx="${default_ixx}" ixy="0" ixz="0" iyy="${default_iyy}" iyz="0" izz="${default_izz}"/>
+	    <inertial>
+			<origin xyz="0 0 0" rpy="0 0 0"/>
+			<mass value="${default_mass}"/>
+			<inertia ixx="${link5_ixx}" ixy="0" ixz="0" iyy="${link5_iyy}" iyz="0" izz="${link5_izz}"/>
 		</inertial>
 		<visual name="VisGeom_Arm_LINK_5">
@@ -509,7 +542,7 @@
 	<link name="Body_Turret">
 		<inertial>
-			<origin xyz="0 0 0" rpy="0 -0 0"/>
-			<mass value="${default_mass}"/>
-			<inertia ixx="${default_ixx}" ixy="0" ixz="0" iyy="${default_iyy}" iyz="0" izz="${default_izz}"/>
+			<origin xyz="0 0 0" rpy="0 0 0"/>
+			<mass value="${turret_mass}"/>
+			<inertia ixx="${turret_ixx}" ixy="0" ixz="0" iyy="${turret_iyy}" iyz="0" izz="${turret_izz}"/>
 		</inertial>
 		<visual name="VisGeom_Turret">
@@ -540,10 +573,10 @@
 		</visual>
 		-->
-		<visual name="VisGeom_AbradingBit">
+		<!--<visual name="VisGeom_AbradingBit">
 			<origin xyz="0.208499 -5.1e-05 -3.438e-05" rpy="0 -0 0"/>
 			<geometry>
 				<mesh filename="package://m2020_urdf_models/rover/meshes/AbradingBitInTurretAtZeroFeed.dae" scale="1 1 1"/>
 			</geometry>
-		</visual>
+		</visual>--> <!-- Commented out TRACLabs -->
 		<!-- hidden visual element
 		<visual name="VisGeom_CoringBit">
@@ -565,7 +598,7 @@
 	<link name="Body_StabilizerFar">
 		<inertial>
-			<origin xyz="-2.5301 0.272349 0.0168656" rpy="0 -0 0"/>
-			<mass value="${default_mass}"/>
-			<inertia ixx="${default_ixx}" ixy="0" ixz="0" iyy="${default_iyy}" iyz="0" izz="${default_izz}"/>
+			<origin xyz="0 0 0" rpy="0 -0 0"/>
+			<mass value="${stabilizer_mass}"/>
+			<inertia ixx="${stabilizer_ixx}" ixy="0" ixz="0" iyy="${stabilizer_iyy}" iyz="0" izz="${stabilizer_izz}"/>
 		</inertial>
 		<visual name="VisGeom_StabilizerFar">
@@ -584,7 +617,7 @@
 	<link name="Body_StabilizerNear">
 		<inertial>
-			<origin xyz="-2.5301 0.272349 0.0168656" rpy="0 -0 0"/>
-			<mass value="${default_mass}"/>
-			<inertia ixx="${default_ixx}" ixy="0" ixz="0" iyy="${default_iyy}" iyz="0" izz="${default_izz}"/>
+			<origin xyz="0 0 0" rpy="0 -0 0"/>
+			<mass value="${stabilizer_mass}"/>
+			<inertia ixx="${stabilizer_ixx}" ixy="0" ixz="0" iyy="${stabilizer_iyy}" iyz="0" izz="${stabilizer_izz}"/>
 		</inertial>
 		<visual name="VisGeom_StabilizerNear">
@@ -603,7 +636,7 @@
 	<link name="Body_WATSON_Cap">
 		<inertial>
-			<origin xyz="-2.6025 0.581204 0.0309103" rpy="0 -0 0"/>
-			<mass value="${default_mass}"/>
-			<inertia ixx="${default_ixx}" ixy="0" ixz="0" iyy="${default_iyy}" iyz="0" izz="${default_izz}"/>
+			<origin xyz="0 0 0" rpy="0 -0 0"/>
+			<mass value="${cap_mass}"/>
+			<inertia ixx="${cap_ixx}" ixy="0" ixz="0" iyy="${cap_iyy}" iyz="0" izz="${cap_izz}"/>
 		</inertial>
 		<visual name="VisGeom_WATSON_Cap">
@@ -622,7 +655,7 @@
 	<link name="Body_SHERLOC_Cap">
 		<inertial>
-			<origin xyz="-2.86084 0.58439 -0.0124626" rpy="0 -0 0"/>
-			<mass value="${default_mass}"/>
-			<inertia ixx="${default_ixx}" ixy="0" ixz="0" iyy="${default_iyy}" iyz="0" izz="${default_izz}"/>
+			<origin xyz="0 0 0" rpy="0 -0 0"/>
+			<mass value="${cap_mass}"/>
+			<inertia ixx="${cap_ixx}" ixy="0" ixz="0" iyy="${cap_iyy}" iyz="0" izz="${cap_izz}"/>
 		</inertial>
 		<visual name="VisGeom_SHERLOC_Cap">
@@ -835,5 +868,5 @@
 		<limit lower="-1.79769e+308" upper="1.79769e+308" effort="1.79769e+308" velocity="1.79769e+308"/>
 	</joint>
-	<joint name="RF_DRIVE" type="fixed"> <!-- TRACLabs Gazebo test hack -->
+	<joint name="RF_DRIVE" type="fixed"> <!-- revolute TRACLabs Gazebo test hack -->
 		<origin xyz="0 0 0" rpy="0 -0 0"/>
 		<parent link="Body_SteerRightFront"/>
@@ -842,12 +875,13 @@
 		<limit lower="-1.79769e+308" upper="1.79769e+308" effort="1.79769e+308" velocity="1.79769e+308"/>
 	</joint>
-	<joint name="RSM_AZ_ENC" type="fixed"> <!-- TRACLabs Gazebo test hack -->
+	<joint name="RSM_AZ_ENC" type="revolute">
 		<origin xyz="0.804037 0.559028 -1.91927" rpy="0 -0 3.12414"/>
 		<parent link="Body_Chassis"/>
 		<child link="Body_RSM_AZ"/>
 		<axis xyz="0 0 1"/>
-		<limit lower="0" upper="6.31809" effort="1.79769e+308" velocity="${head_joint_vel}"/>
-	</joint>
-	<joint name="RSM_EL_ENC" type="fixed"> <!-- TRACLabs Gazebo test hack -->
+		<limit lower="0" upper="6.31809" effort="${head_effort}" velocity="${head_joint_vel}"/>
+		<dynamics damping="${head_damping}" friction="${head_friction}"/>
+	</joint>
+	<joint name="RSM_EL_ENC" type="revolute">
 		<origin xyz="0 0 0" rpy="3.14159 -1.55334 3.14159"/>
 		<parent link="Body_RSM_AZ"/>
@@ -875,38 +909,43 @@
 		<child link="Body_RA_Base"/>
 	</joint>
-	<joint name="JOINT1_ENC" type="fixed"> <!-- TRACLabs Gazebo test hack -->
-		<origin xyz="1.1756 -0.4515 0.3116" rpy="0 -0 0"/>
+	<joint name="JOINT1_ENC" type="revolute">
+		<origin xyz="1.1756 -0.4515 0.3116" rpy="0 0 0"/>
 		<parent link="Body_RA_Base"/>
 		<child link="Body_RA_Link1"/>
 		<axis xyz="0 0 1"/>
-		<limit lower="-3.145" upper="1.592" effort="1.79769e+308" velocity="${arm_joint_vel}"/>
-	</joint>
-	<joint name="JOINT2_ENC" type="fixed"> <!-- TRACLabs Gazebo test hack -->
-		<origin xyz="0.166 0 0" rpy="0 -0 0"/>
+		<limit lower="-3.145" upper="1.592" effort="${arm_default_effort}" velocity="${arm_joint_vel}"/>
+		<dynamics damping="${arm_default_damping}" friction="${arm_default_friction}"/>
+	</joint>
+	<joint name="JOINT2_ENC" type="revolute">
+		<origin xyz="0.166 0 0" rpy="0 0 0"/>
 		<parent link="Body_RA_Link1"/>
 		<child link="Body_RA_Link2"/>
 		<axis xyz="0 -1 0"/>
-		<limit lower="-3.267" upper="0.126" effort="1.79769e+308" velocity="${arm_joint_vel}"/>
-	</joint>
-	<joint name="JOINT3_ENC" type="fixed"> <!-- TRACLabs Gazebo test hack -->
-		<origin xyz="0.8194 0 0" rpy="0 -0 0"/>
+		<limit lower="-3.267" upper="0.126" effort="${arm_default_effort}" velocity="${arm_joint_vel}"/>
+		<dynamics damping="${arm_default_damping}" friction="${arm_default_friction}"/>
+	</joint>
+	<joint name="JOINT3_ENC" type="revolute">
+		<origin xyz="0.8194 0 0" rpy="0 0 0"/>
 		<parent link="Body_RA_Link2"/>
 		<child link="Body_RA_Link3"/>
 		<axis xyz="0 -1 0"/>
-		<limit lower="-2.866" upper="2.866" effort="1.79769e+308" velocity="${arm_joint_vel}"/>
-	</joint>
-	<joint name="JOINT4_ENC" type="fixed"> <!-- TRACLabs Gazebo test hack -->
-		<origin xyz="0.7533 0 0" rpy="0 -0 0"/>
+		<limit lower="-2.866" upper="2.866" effort="${arm_default_effort}" velocity="${arm_joint_vel}"/>
+		<dynamics damping="${arm_default_damping}" friction="${arm_default_friction}"/>
+	</joint>
+	<joint name="JOINT4_ENC" type="revolute">
+		<origin xyz="0.7533 0 0" rpy="0 0 0"/>
 		<parent link="Body_RA_Link3"/>
 		<child link="Body_RA_Link4"/>
 		<axis xyz="0 -1 0"/>
-		<limit lower="-0.178" upper="3.669" effort="1.79769e+308" velocity="${arm_joint_vel}"/>
-	</joint>
-	<joint name="JOINT5_ENC" type="fixed"> <!-- TRACLabs Gazebo test hack -->
-		<origin xyz="-0.1757 0.1791 0" rpy="0 -0 0"/>
+		<limit lower="-0.178" upper="3.669" effort="${arm_default_effort}" velocity="${arm_joint_vel}"/>
+		<dynamics damping="${arm_default_damping}" friction="${arm_default_friction}"/>
+	</joint>
+	<joint name="JOINT5_ENC" type="revolute">
+		<origin xyz="-0.1757 0.1791 0" rpy="0 0 0"/>
 		<parent link="Body_RA_Link4"/>
 		<child link="Body_RA_Link5"/>
 		<axis xyz="0 0 1"/>
-		<limit lower="-0.353" upper="6.636" effort="1.79769e+308" velocity="${arm_joint_vel}"/>
+		<limit lower="-0.353" upper="6.636" effort="${arm_default_effort}" velocity="${arm_joint_vel}"/>
+		<dynamics damping="${arm_default_damping}" friction="${arm_default_friction}"/>
 	</joint>
 	<joint name="JointTurret" type="fixed">
@@ -915,5 +954,5 @@
 		<child link="Body_Turret"/>
 	</joint>
-	<joint name="DRILL_FEED" type="prismatic">
+	<joint name="DRILL_FEED" type="fixed">  <!-- prismatic TRACLabs Gazebo test hack -->
 		<origin xyz="2.5301 -0.272349 -0.0168656" rpy="0 -0 0"/>
 		<parent link="Body_Turret"/>
@@ -922,19 +961,21 @@
 		<limit lower="-1.79769e+308" upper="1.79769e+308" effort="1.79769e+308" velocity="1.79769e+308"/>
 	</joint>
-	<joint name="STABILIZER_LOWER" type="prismatic">
+	<joint name="STABILIZER_LOWER" type="fixed">  <!-- prismatic TRACLabs Gazebo test hack -->
 		<origin xyz="2.5301 -0.272349 -0.0168656" rpy="0 -0 0"/>
 		<parent link="Body_Turret"/>
 		<child link="Body_StabilizerFar"/>
 		<axis xyz="-1 0 0"/>
-		<limit lower="-1.79769e+308" upper="1.79769e+308" effort="1.79769e+308" velocity="1.79769e+308"/>
-	</joint>
-	<joint name="STABILIZER_UPPER" type="prismatic">
+		<limit lower="-1.79769e+308" upper="1.79769e+308" effort="${stabilizer_default_effort}" velocity="${stabilizer_default_vel}"/>
+		<dynamics damping="${arm_default_damping}" friction="${arm_default_friction}"/>
+	</joint>
+	<joint name="STABILIZER_UPPER" type="fixed"> <!-- prismatic TRACLabs Gazebo test hack -->
 		<origin xyz="2.5301 -0.272349 -0.0168656" rpy="0 -0 0"/>
 		<parent link="Body_Turret"/>
 		<child link="Body_StabilizerNear"/>
 		<axis xyz="-1 0 0"/>
-		<limit lower="-1.79769e+308" upper="1.79769e+308" effort="1.79769e+308" velocity="1.79769e+308"/>
-	</joint>
-	<joint name="WATSON_CAP_ENC" type="fixed"> <!-- TRACLabs Gazebo test hack -->
+		<limit lower="-1.79769e+308" upper="1.79769e+308" effort="${stabilizer_default_effort}" velocity="${stabilizer_default_vel}"/>
+		<dynamics damping="${arm_default_damping}" friction="${arm_default_friction}"/>
+	</joint>
+	<joint name="WATSON_CAP_ENC" type="fixed"> <!-- revolute TRACLabs Gazebo test hack -->
 		<origin xyz="2.6025 -0.581204 -0.0309103" rpy="0 -0 0"/>
 		<parent link="Body_Turret"/>
@@ -943,5 +984,5 @@
 		<limit lower="-1.79769e+308" upper="1.79769e+308" effort="1.79769e+308" velocity="1.79769e+308"/>
 	</joint>
-	<joint name="SHERLOC_CAP_ENC" type="fixed"> <!-- TRACLabs Gazebo test hack -->
+	<joint name="SHERLOC_CAP_ENC" type="fixed"> <!-- revolute TRACLabs Gazebo test hack -->
 		<origin xyz="2.86084 -0.58439 0.0124626" rpy="0 -0 0"/>
 		<parent link="Body_Turret"/>

Commit message: tuning persevererence for gazebo

File: urdf/m2020.traclabs.urdf.xacro (robot description, xacro)
@@ -12,5 +12,5 @@
   <xacro:property name="stabilizer_default_vel" value="0.5"/> <!-- original value: 1.79769e+308 -->
   <xacro:property name="stabilizer_default_effort" value="50"/> <!-- original value: 1.79769e+308 -->
-  <xacro:property name="arm_default_damping" value="1.0"/>
+  <xacro:property name="arm_default_damping" value="250.0"/>
   <xacro:property name="arm_default_friction" value="10.0"/>
   <xacro:property name="default_mass" value="3.0" />

Commit message: DAE -> STL   Restored m2020.urdf.xacro and changed m202.traclabs.urdf.xacro

File: urdf/m2020.traclabs.urdf.xacro (robot description, xacro)
@@ -68,5 +68,5 @@
 			<origin xyz="0.09002 0 -1.13338" rpy="0 -0 0"/>
 			<geometry>
-				<mesh filename="package://m2020_urdf_models/rover/meshes/CHASSIS.dae" scale="1 1 1"/>
+				<mesh filename="package://m2020_urdf_models/rover/meshes/low_res/CHASSIS_low_res.stl" scale="1 1 1"/>
 			</geometry>
 		</collision>
@@ -102,5 +102,5 @@
 			<origin xyz="0.142 0 0" rpy="0 -0 0"/>
 			<geometry>
-				<mesh filename="package://m2020_urdf_models/rover/meshes/CenterDifferential.dae" scale="1 1 1"/>
+				<mesh filename="package://m2020_urdf_models/rover/meshes/low_res/CenterDifferential_low_res.stl" scale="1 1 1"/>
 			</geometry>
 		</collision>
@@ -121,5 +121,5 @@
 			<origin xyz="-0.214 0.79959 -0.2405" rpy="0 -0 0"/>
 			<geometry>
-				<mesh filename="package://m2020_urdf_models/rover/meshes/Left_Rocker.dae" scale="1 1 1"/>
+				<mesh filename="package://m2020_urdf_models/rover/meshes/low_res/Left_Rocker_low_res.stl" scale="1 1 1"/>
 			</geometry>
 		</collision>
@@ -140,5 +140,5 @@
 			<origin xyz="0.54 0.91959 -0.4705" rpy="0 -0 0"/>
 			<geometry>
-				<mesh filename="package://m2020_urdf_models/rover/meshes/Left_Bogie.dae" scale="1 1 1"/>
+				<mesh filename="package://m2020_urdf_models/rover/meshes/low_res/Left_Bogie_low_res.stl" scale="1 1 1"/>
 			</geometry>
 		</collision>
@@ -273,5 +273,5 @@
 			<origin xyz="0.54 -0.91959 -0.4705" rpy="0 -0 0"/>
 			<geometry>
-				<mesh filename="package://m2020_urdf_models/rover/meshes/Right_Bogie.dae" scale="1 1 1"/>
+				<mesh filename="package://m2020_urdf_models/rover/meshes/low_res/Right_Bogie_low_res.stl" scale="1 1 1"/>
 			</geometry>
 		</collision>

File: urdf/m2020.urdf.xacro (robot description, xacro)
@@ -22,6 +22,6 @@
 			<origin xyz="0.09002 0 -1.13338" rpy="0 -0 0"/>
 			<geometry>
-				<!--<mesh filename="package://m2020_urdf_models/rover/meshes/CHASSIS.dae" scale="1 1 1"/>-->
-				<mesh filename="package://m2020_urdf_models/rover/meshes/low_res/CHASSIS_low_res.stl" scale="1 1 1"/>
+				<mesh filename="package://m2020_urdf_models/rover/meshes/CHASSIS.dae" scale="1 1 1"/>
+				<!-- <mesh filename="package://m2020_urdf_models/rover/meshes/low_res/CHASSIS_low_res.stl" scale="1 1 1"/> -->
 			</geometry>
 		</visual>
@@ -29,6 +29,6 @@
 			<origin xyz="0.09002 0 -1.13338" rpy="0 -0 0"/>
 			<geometry>
-				<!--<mesh filename="package://m2020_urdf_models/rover/meshes/CHASSIS.dae" scale="1 1 1"/>-->
-				<mesh filename="package://m2020_urdf_models/rover/meshes/low_res/CHASSIS_low_res.stl" scale="1 1 1"/>
+				<mesh filename="package://m2020_urdf_models/rover/meshes/CHASSIS.dae" scale="1 1 1"/>
+				<!-- <mesh filename="package://m2020_urdf_models/rover/meshes/low_res/CHASSIS_low_res.stl" scale="1 1 1"/> -->
 			</geometry>
 		</collision>
@@ -58,6 +58,6 @@
 			<origin xyz="0.142 0 0" rpy="0 -0 0"/>
 			<geometry>
-				<!-- <mesh filename="package://m2020_urdf_models/rover/meshes/CenterDifferential.dae" scale="1 1 1"/> -->
-				<mesh filename="package://m2020_urdf_models/rover/meshes/low_res/CenterDifferential_low_res.stl" scale="1 1 1"/>
+				<mesh filename="package://m2020_urdf_models/rover/meshes/CenterDifferential.dae" scale="1 1 1"/>
+				<!-- <mesh filename="package://m2020_urdf_models/rover/meshes/low_res/CenterDifferential_low_res.stl" scale="1 1 1"/> -->
 			</geometry>
 		</visual>
@@ -72,6 +72,6 @@
 			<origin xyz="-0.214 0.79959 -0.2405" rpy="0 -0 0"/>
 			<geometry>
-				<!-- <mesh filename="package://m2020_urdf_models/rover/meshes/Left_Rocker.dae" scale="1 1 1"/> -->
-				<mesh filename="package://m2020_urdf_models/rover/meshes/low_res/Left_Rocker_low_res.stl" scale="1 1 1"/>
+				<mesh filename="package://m2020_urdf_models/rover/meshes/Left_Rocker.dae" scale="1 1 1"/>
+				<!-- <mesh filename="package://m2020_urdf_models/rover/meshes/low_res/Left_Rocker_low_res.stl" scale="1 1 1"/> -->
 			</geometry>
 		</visual>
@@ -86,6 +86,6 @@
 			<origin xyz="0.54 0.91959 -0.4705" rpy="0 -0 0"/>
 			<geometry>
-				<!-- <mesh filename="package://m2020_urdf_models/rover/meshes/Left_Bogie.dae" scale="1 1 1"/> -->
-				<mesh filename="package://m2020_urdf_models/rover/meshes/low_res/Left_Bogie_low_res.stl" scale="1 1 1"/>
+				<mesh filename="package://m2020_urdf_models/rover/meshes/Left_Bogie.dae" scale="1 1 1"/>
+				<!-- <mesh filename="package://m2020_urdf_models/rover/meshes/low_res/Left_Bogie_low_res.stl" scale="1 1 1"/> -->
 			</geometry>
 		</visual>
@@ -202,6 +202,6 @@
 			<origin xyz="0.54 -0.91959 -0.4705" rpy="0 -0 0"/>
 			<geometry>
-				<!-- <mesh filename="package://m2020_urdf_models/rover/meshes/Right_Bogie.dae" scale="1 1 1"/> -->
-				<mesh filename="package://m2020_urdf_models/rover/meshes/low_res/Right_Bogie_low_res.stl" scale="1 1 1"/>
+				<mesh filename="package://m2020_urdf_models/rover/meshes/Right_Bogie.dae" scale="1 1 1"/>
+				<!-- <mesh filename="package://m2020_urdf_models/rover/meshes/low_res/Right_Bogie_low_res.stl" scale="1 1 1"/> -->
 			</geometry>
 		</visual>
@@ -209,6 +209,6 @@
 			<origin xyz="0.54 -0.91959 -0.4705" rpy="0 -0 0"/>
 			<geometry>
-				<!-- <mesh filename="package://m2020_urdf_models/rover/meshes/Right_Bogie.dae" scale="1 1 1"/> -->
-				<mesh filename="package://m2020_urdf_models/rover/meshes/low_res/Right_Bogie_low_res.stl" scale="1 1 1"/>
+				<mesh filename="package://m2020_urdf_models/rover/meshes/Right_Bogie.dae" scale="1 1 1"/>
+				<!-- <mesh filename="package://m2020_urdf_models/rover/meshes/low_res/Right_Bogie_low_res.stl" scale="1 1 1"/> -->
 			</geometry>
 		</collision>
