Commit message: Converted and decimated eleven more foo.dae files

File: urdf/m2020.traclabs.urdf.xacro (robot description, xacro)
@@ -159,5 +159,5 @@
 			<origin xyz="1.165 1.0625 -0.8705" rpy="0 -0 0"/>
 			<geometry>
-				<mesh filename="package://m2020_urdf_models/rover/meshes/Steer_LeftRear.dae" scale="1 1 1"/>
+				<mesh filename="package://m2020_urdf_models/rover/meshes/low_res/Steer_LeftRear_low_res.stl" scale="1 1 1"/>
 			</geometry>
 		</collision>
@@ -216,5 +216,5 @@
 			<origin xyz="-1.095 1.0625 -0.8705" rpy="0 -0 0"/>
 			<geometry>
-				<mesh filename="package://m2020_urdf_models/rover/meshes/Steer_LeftFront.dae" scale="1 1 1"/>
+				<mesh filename="package://m2020_urdf_models/rover/meshes/low_res/Steer_LeftFront_low_res.stl" scale="1 1 1"/>
 			</geometry>
 		</collision>
@@ -254,5 +254,5 @@
 			<origin xyz="-0.214 -0.79959 -0.2405" rpy="0 -0 0"/>
 			<geometry>
-				<mesh filename="package://m2020_urdf_models/rover/meshes/Right_Rocker.dae" scale="1 1 1"/>
+				<mesh filename="package://m2020_urdf_models/rover/meshes/low_res/Right_Rocker_low_res.stl" scale="1 1 1"/>
 			</geometry>
 		</collision>
@@ -292,5 +292,5 @@
 			<origin xyz="1.165 -1.0625 -0.8705" rpy="0 -0 0"/>
 			<geometry>
-				<mesh filename="package://m2020_urdf_models/rover/meshes/Steer_RightRear.dae" scale="1 1 1"/>
+				<mesh filename="package://m2020_urdf_models/rover/meshes/low_res/Steer_RightRear_low_res.stl" scale="1 1 1"/>
 			</geometry>
 		</collision>
@@ -349,5 +349,5 @@
 			<origin xyz="-1.095 -1.0625 -0.8705" rpy="0 -0 0"/>
 			<geometry>
-				<mesh filename="package://m2020_urdf_models/rover/meshes/Steer_RightFront.dae" scale="1 1 1"/>
+				<mesh filename="package://m2020_urdf_models/rover/meshes/low_res/Steer_RightFront_low_res.stl" scale="1 1 1"/>
 			</geometry>
 		</collision>
@@ -387,5 +387,5 @@
 			<origin xyz="-0.714017 -0.559028 0.78589" rpy="0 -0 0"/>
 			<geometry>
-				<mesh filename="package://m2020_urdf_models/rover/meshes/RSM.dae" scale="1 1 1"/>
+				<mesh filename="package://m2020_urdf_models/rover/meshes/low_res/RSM_low_res.stl" scale="1 1 1"/>
 			</geometry>
 		</collision>
@@ -406,5 +406,5 @@
 			<origin xyz="-0.714017 -0.559028 0.78589" rpy="0 -0 0"/>
 			<geometry>
-				<mesh filename="package://m2020_urdf_models/rover/meshes/RSM_Head.dae" scale="1 1 1"/>
+				<mesh filename="package://m2020_urdf_models/rover/meshes/low_res/RSM_Head_low_res.stl" scale="1 1 1"/>
 			</geometry>
 		</collision>
@@ -425,5 +425,5 @@
 			<origin xyz="0.46 0.475 -0.0005" rpy="0 -0 0"/>
 			<geometry>
-				<mesh filename="package://m2020_urdf_models/rover/meshes/HGA_AZ.dae" scale="1 1 1"/>
+				<mesh filename="package://m2020_urdf_models/rover/meshes/low_res/HGA_AZ_low_res.stl" scale="1 1 1"/>
 			</geometry>
 		</collision>
@@ -444,5 +444,5 @@
 			<origin xyz="0.46 0.475 0.2475" rpy="0 -0 0"/>
 			<geometry>
-				<mesh filename="package://m2020_urdf_models/rover/meshes/HGA_EL.dae" scale="1 1 1"/>
+				<mesh filename="package://m2020_urdf_models/rover/meshes/low_res/HGA_EL_low_res.stl" scale="1 1 1"/>
 			</geometry>
 		</collision>
@@ -470,5 +470,5 @@
 			<origin xyz="-1.1756 0.4515 -0.3116" rpy="0 -0 0"/>
 			<geometry>
-				<mesh filename="package://m2020_urdf_models/rover/meshes/Arm_LINK_1.dae" scale="1 1 1"/>
+				<mesh filename="package://m2020_urdf_models/rover/meshes/low_res/Arm_LINK_1_low_res.stl" scale="1 1 1"/>
 			</geometry>
 		</collision>
@@ -489,5 +489,7 @@
 			<origin xyz="-1.3416 0.4515 -0.3116" rpy="0 -0 0"/>
 			<geometry>
-				<mesh filename="package://m2020_urdf_models/rover/meshes/Arm_LINK_2.dae" scale="1 1 1"/>
+				<!-- todo -->
+				<!-- <mesh filename="package://m2020_urdf_models/rover/meshes/Arm_LINK_2.dae" scale="1 1 1"/> -->
+				<mesh filename="package://m2020_urdf_models/rover/meshes/low_res/Arm_LINK_2_low_res.stl" scale="1 1 1"/>
 			</geometry>
 		</collision>

Commit message: Added eight more STL files. Now only the Wheels remain

File: urdf/m2020.traclabs.urdf.xacro (robot description, xacro)
@@ -489,6 +489,4 @@
 			<origin xyz="-1.3416 0.4515 -0.3116" rpy="0 -0 0"/>
 			<geometry>
-				<!-- todo -->
-				<!-- <mesh filename="package://m2020_urdf_models/rover/meshes/Arm_LINK_2.dae" scale="1 1 1"/> -->
 				<mesh filename="package://m2020_urdf_models/rover/meshes/low_res/Arm_LINK_2_low_res.stl" scale="1 1 1"/>
 			</geometry>
@@ -510,5 +508,5 @@
 			<origin xyz="-2.161 0.4515 -0.3116" rpy="0 -0 0"/>
 			<geometry>
-				<mesh filename="package://m2020_urdf_models/rover/meshes/Arm_LINK_3.dae" scale="1 1 1"/>
+				<mesh filename="package://m2020_urdf_models/rover/meshes/low_res/Arm_LINK_3_low_res.stl" scale="1 1 1"/>
 			</geometry>
 		</collision>
@@ -529,5 +527,5 @@
 			<origin xyz="-2.9143 0.4515 -0.3116" rpy="0 -0 0"/>
 			<geometry>
-				<mesh filename="package://m2020_urdf_models/rover/meshes/Arm_LINK_4.dae" scale="1 1 1"/>
+				<mesh filename="package://m2020_urdf_models/rover/meshes/low_res/Arm_LINK_4_low_res.stl" scale="1 1 1"/>
 			</geometry>
 		</collision>
@@ -548,5 +546,5 @@
 			<origin xyz="-2.7386 0.2724 -0.3116" rpy="0 -0 0"/>
 			<geometry>
-				<mesh filename="package://m2020_urdf_models/rover/meshes/Arm_LINK_5.dae" scale="1 1 1"/>
+				<mesh filename="package://m2020_urdf_models/rover/meshes/low_res/Arm_LINK_5_low_res.stl" scale="1 1 1"/>
 			</geometry>
 		</collision>
@@ -567,5 +565,5 @@
 			<origin xyz="0 0 0" rpy="0 -0 0"/>
 			<geometry>
-				<mesh filename="package://m2020_urdf_models/rover/meshes/Turret.dae" scale="1 1 1"/>
+				<mesh filename="package://m2020_urdf_models/rover/meshes/low_res/Turret_low_res.stl" scale="1 1 1"/>
 			</geometry>
 		</collision>
@@ -623,5 +621,5 @@
 			<origin xyz="0.208499 -5.1e-05 -3.438e-05" rpy="0 -0 0"/>
 			<geometry>
-				<mesh filename="package://m2020_urdf_models/rover/meshes/StabilizerFarInTurret.dae" scale="1 1 1"/>
+				<mesh filename="package://m2020_urdf_models/rover/meshes/low_res/StabilizerFarInTurret_low_res.stl" scale="1 1 1"/>
 			</geometry>
 		</collision>
@@ -642,5 +640,5 @@
 			<origin xyz="0.208499 -5.1e-05 -3.438e-05" rpy="0 -0 0"/>
 			<geometry>
-				<mesh filename="package://m2020_urdf_models/rover/meshes/StabilizerNearInTurret.dae" scale="1 1 1"/>
+				<mesh filename="package://m2020_urdf_models/rover/meshes/low_res/StabilizerNearInTurret_low_res.stl" scale="1 1 1"/>
 			</geometry>
 		</collision>
@@ -661,5 +659,5 @@
 			<origin xyz="-2.6025 0.581204 0.0309103" rpy="0 -0 0"/>
 			<geometry>
-				<mesh filename="package://m2020_urdf_models/rover/meshes/WATSON_Camera_Cap.dae" scale="1 1 1"/>
+				<mesh filename="package://m2020_urdf_models/rover/meshes/low_res/WATSON_Camera_Cap_low_res.stl" scale="1 1 1"/>
 			</geometry>
 		</collision>
@@ -680,5 +678,5 @@
 			<origin xyz="-2.86084 0.58439 -0.0124626" rpy="0 -0 0"/>
 			<geometry>
-				<mesh filename="package://m2020_urdf_models/rover/meshes/ContextImager_Cap.dae" scale="1 1 1"/>
+				<mesh filename="package://m2020_urdf_models/rover/meshes/low_res/ContextImager_Cap_low_res.stl" scale="1 1 1"/>
 			</geometry>
 		</collision>
