Commit message: Added files for ingenuity

File: urdf/mhs.urdf.xacro (robot description, xacro)
@@ -2,5 +2,6 @@
 <!-- This file was generated automatically. [2020_07_14_13_00_00] -->
 <!-- [Tool url: git@github.jpl.nasa.gov:CR/rst.git, branch: dev/working, commit_hash: c6befd6c, commit_time: 2020-07-13 19:17:50 -0700] -->
-<robot name="ingenuity">
+<robot name="ingenuity" xmlns:xacro="http://www.ros.org/wiki/xacro">
+  <xacro:property name="leg_joint_vel" value="0.2" /> <!-- original value: 1.79769e+308 . TRACLabs edit -->
 	<link name="root">
 		<inertial>
@@ -154,5 +155,5 @@
 		<child link="Body_Joint_Leg02_Axis"/>
 		<axis xyz="-1 0 0"/>
-		<limit lower="-1.79769e+308" upper="1.79769e+308" effort="1.79769e+308" velocity="1.79769e+308"/>
+		<limit lower="-1.79769e+308" upper="1.79769e+308" effort="1.79769e+308" velocity="${leg_joint_vel}"/>
 	</joint>
 	<joint name="MHS_Leg02_v16" type="fixed">
@@ -166,5 +167,5 @@
 		<child link="Body_Joint_Leg01_Axis"/>
 		<axis xyz="-1 0 0"/>
-		<limit lower="-1.79769e+308" upper="1.79769e+308" effort="1.79769e+308" velocity="1.79769e+308"/>
+		<limit lower="-1.79769e+308" upper="1.79769e+308" effort="1.79769e+308" velocity="${leg_joint_vel}"/>
 	</joint>
 	<joint name="MHS_Leg01_v16" type="fixed">
@@ -178,5 +179,5 @@
 		<child link="Body_Joint_Leg03_Axis"/>
 		<axis xyz="-1 0 0"/>
-		<limit lower="-1.79769e+308" upper="1.79769e+308" effort="1.79769e+308" velocity="1.79769e+308"/>
+		<limit lower="-1.79769e+308" upper="1.79769e+308" effort="1.79769e+308" velocity="${leg_joint_vel}"/>
 	</joint>
 	<joint name="MHS_Leg03_v16" type="fixed">
@@ -190,5 +191,5 @@
 		<child link="Body_Joint_Leg04_Axis"/>
 		<axis xyz="-1 0 0"/>
-		<limit lower="-1.79769e+308" upper="1.79769e+308" effort="1.79769e+308" velocity="1.79769e+308"/>
+		<limit lower="-1.79769e+308" upper="1.79769e+308" effort="1.79769e+308" velocity="${leg_joint_vel}"/>
 	</joint>
 	<joint name="MHS_Leg04_v16" type="fixed">
@@ -197,5 +198,5 @@
 		<child link="Body_MHS_Leg04_v16"/>
 	</joint>
-	<joint name="MHS_NAVCAM">
+	<joint name="MHS_NAVCAM" type="fixed"> <!-- TRACLabs note: Added type=fixed to the original, which didn't have a type -->
 		<origin xyz="0.0 0.0616891 0.13743" rpy="-0.0027478 0.0580433 -1.57391594"/>
 		<parent link="Body_MHS_MainBody_v16"/>

Commit message: Added base frame for legs group of ingenuity, otherwise IC goes angry and nav IM disappears. Go figure

File: urdf/mhs.urdf.xacro (robot description, xacro)
@@ -69,4 +69,10 @@
 			</geometry>
 		</visual>
+		<collision name="ColGeom_MHS_Leg02_v16">
+			<origin xyz="0 0 0" rpy="0 -0 0"/>
+			<geometry>
+				<mesh filename="package://m2020_urdf_models/mhs/meshes/MHS_Leg02_v16.dae" scale="1 1 1"/>
+			</geometry>
+		</collision>
 	</link>
 	<link name="Body_Joint_Leg01_Axis">
@@ -89,4 +95,10 @@
 			</geometry>
 		</visual>
+		<collision name="ColGeom_MHS_Leg01_v16">
+			<origin xyz="0 0 0" rpy="0 -0 0"/>
+			<geometry>
+				<mesh filename="package://m2020_urdf_models/mhs/meshes/MHS_Leg01_v16.dae" scale="1 1 1"/>
+			</geometry>
+		</collision>
 	</link>
 	<link name="Body_Joint_Leg03_Axis">
@@ -109,4 +121,10 @@
 			</geometry>
 		</visual>
+		<collision name="ColGeom_MHS_Leg03_v16">
+			<origin xyz="0 0 0" rpy="0 -0 0"/>
+			<geometry>
+				<mesh filename="package://m2020_urdf_models/mhs/meshes/MHS_Leg03_v16.dae" scale="1 1 1"/>
+			</geometry>
+		</collision>
 	</link>
 	<link name="Body_Joint_Leg04_Axis">
@@ -129,4 +147,10 @@
 			</geometry>
 		</visual>
+		<collision name="ColGeom_MHS_Leg04_v16">
+			<origin xyz="0 0 0" rpy="0 -0 0"/>
+			<geometry>
+				<mesh filename="package://m2020_urdf_models/mhs/meshes/MHS_Leg04_v16.dae" scale="1 1 1"/>
+			</geometry>
+		</collision>
 	</link>
 	<link name="Frame_MHS_NAVCAM"></link>

Commit message: flipped Z-axis to be up

File: urdf/mhs.urdf.xacro (robot description, xacro)
@@ -6,5 +6,5 @@
 	<link name="root">
 		<inertial>
-			<origin xyz="0 0 0" rpy="0 -0 0"/>
+			<origin xyz="0 0 0" rpy="0 0 0"/>
 			<mass value="0"/>
 			<inertia ixx="0" ixy="0" ixz="0" iyy="0" iyz="0" izz="0"/>
@@ -156,5 +156,5 @@
 	<link name="Frame_MHS_NAVCAM"></link>
 	<joint name="MHS_MainBody_v16" type="fixed">
-		<origin xyz="0 0 0" rpy="0 -0 0"/>
+		<origin xyz="0 0 0" rpy="3.14 0 0"/>
 		<parent link="root"/>
 		<child link="Body_MHS_MainBody_v16"/>

Commit message: adding missing collision meshes for ingenuity

File: urdf/mhs.urdf.xacro (robot description, xacro)
@@ -23,4 +23,10 @@
 			</geometry>
 		</visual>
+		<collision name="ColGeom_MHS_MainBody_v16">
+			<origin xyz="0 0 0" rpy="0 -0 0"/>
+			<geometry>
+				<mesh filename="package://m2020_urdf_models/mhs/meshes/MHS_MainBody_v16.dae" scale="1 1 1"/>
+			</geometry>
+		</collision>
 	</link>
 	<link name="Body_MHS_TopBlades_v16">
@@ -36,5 +42,11 @@
 			</geometry>
 		</visual>
-	</link>
+		<collision name="ColGeom_MHS_TopBlades_v16">
+			<origin xyz="0 0 0" rpy="0 -0 0"/>
+			<geometry>
+				<mesh filename="package://m2020_urdf_models/mhs/meshes/MHS_TopBlades_v16.dae" scale="1 1 1"/>
+			</geometry>
+		</collision>
+  </link>
 	<link name="Body_MHS_BottomBlades_v16">
 		<inertial>
@@ -49,5 +61,11 @@
 			</geometry>
 		</visual>
-	</link>
+    <collision name="ColGeom_MHS_BottomBlades_v16">
+			<origin xyz="0 0 0" rpy="0 -0 0"/>
+			<geometry>
+				<mesh filename="package://m2020_urdf_models/mhs/meshes/MHS_BottomBlades_v16.dae" scale="1 1 1"/>
+			</geometry>
+		</collision>
+  </link>
 	<link name="Body_Joint_Leg02_Axis">
 		<inertial>

Commit message: replacing added meshes with large simplified collision model

File: urdf/mhs.urdf.xacro (robot description, xacro)
@@ -25,7 +25,7 @@
 		<collision name="ColGeom_MHS_MainBody_v16">
 			<origin xyz="0 0 0" rpy="0 -0 0"/>
-			<geometry>
-				<mesh filename="package://m2020_urdf_models/mhs/meshes/MHS_MainBody_v16.dae" scale="1 1 1"/>
-			</geometry>
+      <geometry>
+        <box size="1.22 1.22 0.55" />
+      </geometry>
 		</collision>
 	</link>
@@ -42,10 +42,4 @@
 			</geometry>
 		</visual>
-		<collision name="ColGeom_MHS_TopBlades_v16">
-			<origin xyz="0 0 0" rpy="0 -0 0"/>
-			<geometry>
-				<mesh filename="package://m2020_urdf_models/mhs/meshes/MHS_TopBlades_v16.dae" scale="1 1 1"/>
-			</geometry>
-		</collision>
   </link>
 	<link name="Body_MHS_BottomBlades_v16">
@@ -61,10 +55,4 @@
 			</geometry>
 		</visual>
-    <collision name="ColGeom_MHS_BottomBlades_v16">
-			<origin xyz="0 0 0" rpy="0 -0 0"/>
-			<geometry>
-				<mesh filename="package://m2020_urdf_models/mhs/meshes/MHS_BottomBlades_v16.dae" scale="1 1 1"/>
-			</geometry>
-		</collision>
   </link>
 	<link name="Body_Joint_Leg02_Axis">

Commit message: setting up ingenuity for gazebo

File: urdf/mhs.urdf.xacro (robot description, xacro)
@@ -7,6 +7,6 @@
 		<inertial>
 			<origin xyz="0 0 0" rpy="0 0 0"/>
-			<mass value="0"/>
-			<inertia ixx="0" ixy="0" ixz="0" iyy="0" iyz="0" izz="0"/>
+			<mass value="0.1"/>
+			<inertia ixx="0.001" ixy="0" ixz="0" iyy="0.001" iyz="0" izz="0.001"/>
 		</inertial>
 	</link>
@@ -14,6 +14,6 @@
 		<inertial>
 			<origin xyz="0 0 0" rpy="0 -0 0"/>
-			<mass value="0"/>
-			<inertia ixx="0" ixy="0" ixz="0" iyy="0" iyz="0" izz="0"/>
+			<mass value="10"/>
+			<inertia ixx="0.001" ixy="0" ixz="0" iyy="0.001" iyz="0" izz="0.001"/>
 		</inertial>
 		<visual name="VisGeom_MHS_MainBody_v16">
@@ -25,7 +25,10 @@
 		<collision name="ColGeom_MHS_MainBody_v16">
 			<origin xyz="0 0 0" rpy="0 -0 0"/>
-      <geometry>
+<!--       <geometry>
         <box size="1.22 1.22 0.55" />
-      </geometry>
+      </geometry> -->
+			<geometry>
+				<mesh filename="package://m2020_urdf_models/mhs/meshes/MHS_MainBody_v16.dae" scale="1 1 1"/>
+			</geometry>
 		</collision>
 	</link>
@@ -33,6 +36,6 @@
 		<inertial>
 			<origin xyz="0 0 0" rpy="0 -0 0"/>
-			<mass value="0"/>
-			<inertia ixx="0" ixy="0" ixz="0" iyy="0" iyz="0" izz="0"/>
+			<mass value="0.1"/>
+			<inertia ixx="0.001" ixy="0" ixz="0" iyy="0.001" iyz="0" izz="0.001"/>
 		</inertial>
 		<visual name="VisGeom_MHS_TopBlades_v16">
@@ -46,6 +49,6 @@
 		<inertial>
 			<origin xyz="0 0 0" rpy="0 -0 0"/>
-			<mass value="0"/>
-			<inertia ixx="0" ixy="0" ixz="0" iyy="0" iyz="0" izz="0"/>
+			<mass value="0.1"/>
+			<inertia ixx="0.001" ixy="0" ixz="0" iyy="0.001" iyz="0" izz="0.001"/>
 		</inertial>
 		<visual name="VisGeom_MHS_BottomBlades_v16">
@@ -59,6 +62,6 @@
 		<inertial>
 			<origin xyz="0 0 0" rpy="0 -0 0"/>
-			<mass value="0"/>
-			<inertia ixx="0" ixy="0" ixz="0" iyy="0" iyz="0" izz="0"/>
+			<mass value="0.1"/>
+			<inertia ixx="0.001" ixy="0" ixz="0" iyy="0.001" iyz="0" izz="0.001"/>
 		</inertial>
 	</link>
@@ -66,6 +69,6 @@
 		<inertial>
 			<origin xyz="0 0 0" rpy="0 -0 0"/>
-			<mass value="0"/>
-			<inertia ixx="0" ixy="0" ixz="0" iyy="0" iyz="0" izz="0"/>
+			<mass value="0.1"/>
+			<inertia ixx="0.001" ixy="0" ixz="0" iyy="0.001" iyz="0" izz="0.001"/>
 		</inertial>
 		<visual name="VisGeom_MHS_Leg02_v16">
@@ -85,6 +88,6 @@
 		<inertial>
 			<origin xyz="0 0 0" rpy="0 -0 0"/>
-			<mass value="0"/>
-			<inertia ixx="0" ixy="0" ixz="0" iyy="0" iyz="0" izz="0"/>
+			<mass value="0.1"/>
+			<inertia ixx="0.001" ixy="0" ixz="0" iyy="0.001" iyz="0" izz="0.001"/>
 		</inertial>
 	</link>
@@ -92,6 +95,6 @@
 		<inertial>
 			<origin xyz="0 0 0" rpy="0 -0 0"/>
-			<mass value="0"/>
-			<inertia ixx="0" ixy="0" ixz="0" iyy="0" iyz="0" izz="0"/>
+			<mass value="0.1"/>
+			<inertia ixx="0.001" ixy="0" ixz="0" iyy="0.001" iyz="0" izz="0.001"/>
 		</inertial>
 		<visual name="VisGeom_MHS_Leg01_v16">
@@ -111,6 +114,6 @@
 		<inertial>
 			<origin xyz="0 0 0" rpy="0 -0 0"/>
-			<mass value="0"/>
-			<inertia ixx="0" ixy="0" ixz="0" iyy="0" iyz="0" izz="0"/>
+			<mass value="0.1"/>
+			<inertia ixx="0.001" ixy="0" ixz="0" iyy="0.001" iyz="0" izz="0.001"/>
 		</inertial>
 	</link>
@@ -118,6 +121,6 @@
 		<inertial>
 			<origin xyz="0 0 0" rpy="0 -0 0"/>
-			<mass value="0"/>
-			<inertia ixx="0" ixy="0" ixz="0" iyy="0" iyz="0" izz="0"/>
+			<mass value="0.1"/>
+			<inertia ixx="0.001" ixy="0" ixz="0" iyy="0.001" iyz="0" izz="0.001"/>
 		</inertial>
 		<visual name="VisGeom_MHS_Leg03_v16">
@@ -137,6 +140,6 @@
 		<inertial>
 			<origin xyz="0 0 0" rpy="0 -0 0"/>
-			<mass value="0"/>
-			<inertia ixx="0" ixy="0" ixz="0" iyy="0" iyz="0" izz="0"/>
+			<mass value="0.1"/>
+			<inertia ixx="0.001" ixy="0" ixz="0" iyy="0.001" iyz="0" izz="0.001"/>
 		</inertial>
 	</link>
@@ -144,6 +147,6 @@
 		<inertial>
 			<origin xyz="0 0 0" rpy="0 -0 0"/>
-			<mass value="0"/>
-			<inertia ixx="0" ixy="0" ixz="0" iyy="0" iyz="0" izz="0"/>
+			<mass value="0.1"/>
+			<inertia ixx="0.001" ixy="0" ixz="0" iyy="0.001" iyz="0" izz="0.001"/>
 		</inertial>
 		<visual name="VisGeom_MHS_Leg04_v16">
@@ -166,17 +169,17 @@
 		<child link="Body_MHS_MainBody_v16"/>
 	</joint>
-	<joint name="MHS_TopBlades_v16" type="revolute">
+	<joint name="MHS_TopBlades_v16" type="continuous">
 		<origin xyz="0 0 0" rpy="0 -0 0"/>
 		<parent link="Body_MHS_MainBody_v16"/>
 		<child link="Body_MHS_TopBlades_v16"/>
 		<axis xyz="0 0 1"/>
-		<limit lower="-1.79769e+308" upper="1.79769e+308" effort="1.79769e+308" velocity="1.79769e+308"/>
-	</joint>
-	<joint name="MHS_BottomBlades_v16" type="revolute">
+		<limit effort="1.79769e+308" velocity="1.79769e+308"/>
+	</joint>
+	<joint name="MHS_BottomBlades_v16" type="continuous">
 		<origin xyz="0 0 0" rpy="0 -0 0.994839"/>
 		<parent link="Body_MHS_MainBody_v16"/>
 		<child link="Body_MHS_BottomBlades_v16"/>
 		<axis xyz="0 0 1"/>
-		<limit lower="-1.79769e+308" upper="1.79769e+308" effort="1.79769e+308" velocity="1.79769e+308"/>
+		<limit effort="1.79769e+308" velocity="1.79769e+308"/>
 	</joint>
 	<joint name="Joint_Leg02_Axis" type="revolute">
